Commit message: Use 3D lidar ring for simulated laser scan

File: ros2_ws/src/scout_description/urdf/accessories/vlp16_mount.urdf.xacro (robot description, xacro)
@@ -9,7 +9,9 @@
       topic
       robot_namespace:=/
-      update_rate:=5
-      horizontal_samples:=360
+      update_rate:=10
+      horizontal_samples:=720
       vertical_samples:=16
+      min_vertical_angle:=-0.2792526803190927
+      max_vertical_angle:=0.24434609527920614
       min_range:=0.3
       max_range:=25.0
@@ -69,4 +71,6 @@
       lasers="${vertical_samples}"
       samples="${horizontal_samples}"
+      min_vertical_angle="${min_vertical_angle}"
+      max_vertical_angle="${max_vertical_angle}"
       collision_range="${min_range}"
       min_range="${min_range}"

File: ros2_ws/src/scout_description/urdf/scout.urdf.xacro (robot description, xacro)
@@ -29,6 +29,6 @@
     <xacro:arg name="laser_3d_rpy" default="$(optenv SCOUT_LASER_3D_RPY 0 0 0)" />
     <xacro:arg name="laser_3d_topic" default="$(optenv SCOUT_LASER_3D_TOPIC points)" />
-    <xacro:arg name="laser_3d_update_rate" default="$(optenv SCOUT_LASER_3D_UPDATE_RATE 5)" />
-    <xacro:arg name="laser_3d_horizontal_samples" default="$(optenv SCOUT_LASER_3D_HORIZONTAL_SAMPLES 360)" />
+    <xacro:arg name="laser_3d_update_rate" default="$(optenv SCOUT_LASER_3D_UPDATE_RATE 10)" />
+    <xacro:arg name="laser_3d_horizontal_samples" default="$(optenv SCOUT_LASER_3D_HORIZONTAL_SAMPLES 720)" />
     <xacro:arg name="laser_3d_vertical_samples" default="$(optenv SCOUT_LASER_3D_VERTICAL_SAMPLES 16)" />
     <xacro:arg name="laser_3d_min_range" default="$(optenv SCOUT_LASER_3D_MIN_RANGE 0.3)" />

File: ros2_ws/src/velodyne_simulator/velodyne_description/urdf/VLP-16.urdf.xacro (robot description, xacro)
@@ -2,5 +2,5 @@
 <robot xmlns:xacro="http://www.ros.org/wiki/xacro" name="VLP-16">
   <xacro:property name="M_PI" value="3.1415926535897931" />
-  <xacro:macro name="VLP-16" params="*origin parent:=base_link name:=velodyne tf_prefix:='' topic:=/velodyne_points organize_cloud:=false hz:=10 lasers:=16 samples:=1875 collision_range:=0.3 min_range:=0.9 max_range:=130.0 noise:=0.008 min_angle:=-${M_PI} max_angle:=${M_PI} gpu:=false">
+  <xacro:macro name="VLP-16" params="*origin parent:=base_link name:=velodyne tf_prefix:='' topic:=/velodyne_points organize_cloud:=false hz:=10 lasers:=16 samples:=1875 collision_range:=0.3 min_range:=0.9 max_range:=130.0 noise:=0.008 min_angle:=-${M_PI} max_angle:=${M_PI} min_vertical_angle:=-${15.0*M_PI/180.0} max_vertical_angle:=${15.0*M_PI/180.0} gpu:=false">
     <joint name="${name}_base_mount_joint" type="fixed">
       <xacro:insert_block name="origin" />
@@ -74,6 +74,6 @@
                 <samples>${lasers}</samples>
                 <resolution>1</resolution>
-                <min_angle>-${15.0*M_PI/180.0}</min_angle>
-                <max_angle> ${15.0*M_PI/180.0}</max_angle>
+                <min_angle>${min_vertical_angle}</min_angle>
+                <max_angle>${max_vertical_angle}</max_angle>
               </vertical>
             </scan>
@@ -119,6 +119,6 @@
                 <samples>${lasers}</samples>
                 <resolution>1</resolution>
-                <min_angle>-${15.0*M_PI/180.0}</min_angle>
-                <max_angle> ${15.0*M_PI/180.0}</max_angle>
+                <min_angle>${min_vertical_angle}</min_angle>
+                <max_angle>${max_vertical_angle}</max_angle>
               </vertical>
             </scan>
