Commit message: Add FAST-LIVO2 Ackermann MPPI simulation

File: ros2_ws/src/agribot_ackermann_mppi/urdf/ackermann_scout.urdf.xacro (robot description, xacro)
@@ -88,4 +88,16 @@
     <child link="imu_link" />
   </joint>
+  <link name="camera_realsense"/>
+  <joint name="camera_realsense_joint" type="fixed">
+    <origin xyz="0.025 0 0.42" rpy="0 0 0" />
+    <parent link="base_link" />
+    <child link="camera_realsense" />
+  </joint>
+  <link name="camera_realsense_gazebo"/>
+  <joint name="camera_realsense_gazebo_joint" type="fixed">
+    <origin xyz="0 0 0" rpy="${-M_PI/2} 0 ${-M_PI/2}" />
+    <parent link="camera_realsense" />
+    <child link="camera_realsense_gazebo" />
+  </joint>
   <xacro:ackermann_wheel_link wheel_prefix="front_left" is_right="false" />
   <xacro:ackermann_wheel_link wheel_prefix="front_right" is_right="true" />
@@ -207,4 +219,6 @@
   <xacro:disable_gravity ref="vlp16_base_link" />
   <xacro:disable_gravity ref="vlp16" />
+  <xacro:disable_gravity ref="camera_realsense" />
+  <xacro:disable_gravity ref="camera_realsense_gazebo" />
   <gazebo reference="front_left_wheel_link">
     <mu1>1.8</mu1>

Commit message: 移除FAST-LIVO2及专属依赖

File: ros2_ws/src/agribot_ackermann_mppi/urdf/ackermann_scout.urdf.xacro (robot description, xacro)
@@ -88,16 +88,4 @@
     <child link="imu_link" />
   </joint>
-  <link name="camera_realsense"/>
-  <joint name="camera_realsense_joint" type="fixed">
-    <origin xyz="0.025 0 0.42" rpy="0 0 0" />
-    <parent link="base_link" />
-    <child link="camera_realsense" />
-  </joint>
-  <link name="camera_realsense_gazebo"/>
-  <joint name="camera_realsense_gazebo_joint" type="fixed">
-    <origin xyz="0 0 0" rpy="${-M_PI/2} 0 ${-M_PI/2}" />
-    <parent link="camera_realsense" />
-    <child link="camera_realsense_gazebo" />
-  </joint>
   <xacro:ackermann_wheel_link wheel_prefix="front_left" is_right="false" />
   <xacro:ackermann_wheel_link wheel_prefix="front_right" is_right="true" />
@@ -219,6 +207,4 @@
   <xacro:disable_gravity ref="vlp16_base_link" />
   <xacro:disable_gravity ref="vlp16" />
-  <xacro:disable_gravity ref="camera_realsense" />
-  <xacro:disable_gravity ref="camera_realsense_gazebo" />
   <gazebo reference="front_left_wheel_link">
     <mu1>1.8</mu1>

Commit message: feat: add four-camera BEV perception pipeline

File: ros2_ws/src/agribot_ackermann_mppi/urdf/ackermann_scout.urdf.xacro (robot description, xacro)
@@ -20,4 +20,7 @@
   <xacro:property name="wheel_radius" value="1.6459e-01" />
   <xacro:property name="wheel_joint_friction" value="20.0" />
+  <xacro:property name="bev_camera_radius" value="0.09" />
+  <xacro:property name="bev_camera_height" value="0.76521" />
+  <xacro:property name="bev_camera_pitch" value="0.436332" />
   <xacro:macro name="ackermann_wheel_link" params="wheel_prefix is_right">
     <link name="${wheel_prefix}_wheel_link">
@@ -51,4 +54,28 @@
     </gazebo>
   </xacro:macro>
+  <xacro:macro name="bev_camera_frame" params="name xyz yaw">
+    <link name="${name}_camera_link">
+      <visual>
+        <origin xyz="0 0 0" rpy="0 0 0" />
+        <geometry>
+          <box size="0.05 0.035 0.035" />
+        </geometry>
+        <material name="${name}_camera_dark">
+          <color rgba="0.08 0.08 0.08 1.0" />
+        </material>
+      </visual>
+    </link>
+    <joint name="${name}_camera_joint" type="fixed">
+      <origin xyz="${xyz}" rpy="0 ${bev_camera_pitch} ${yaw}" />
+      <parent link="base_link" />
+      <child link="${name}_camera_link" />
+    </joint>
+    <link name="${name}_camera_optical_frame" />
+    <joint name="${name}_camera_optical_joint" type="fixed">
+      <origin xyz="0 0 0" rpy="${-M_PI/2} 0 ${-M_PI/2}" />
+      <parent link="${name}_camera_link" />
+      <child link="${name}_camera_optical_frame" />
+    </joint>
+  </xacro:macro>
   <link name="base_link">
     <inertial>
@@ -88,4 +115,12 @@
     <child link="imu_link" />
   </joint>
+  <xacro:bev_camera_frame
+    name="bev_front" xyz="${bev_camera_radius} 0 ${bev_camera_height}" yaw="0" />
+  <xacro:bev_camera_frame
+    name="bev_left" xyz="0 ${bev_camera_radius} ${bev_camera_height}" yaw="${M_PI/2}" />
+  <xacro:bev_camera_frame
+    name="bev_rear" xyz="${-bev_camera_radius} 0 ${bev_camera_height}" yaw="${M_PI}" />
+  <xacro:bev_camera_frame
+    name="bev_right" xyz="0 ${-bev_camera_radius} ${bev_camera_height}" yaw="${-M_PI/2}" />
   <xacro:ackermann_wheel_link wheel_prefix="front_left" is_right="false" />
   <xacro:ackermann_wheel_link wheel_prefix="front_right" is_right="true" />

Commit message: 完善阿克曼融合定位与长距离航点仿真

File: ros2_ws/src/agribot_ackermann_mppi/urdf/ackermann_scout.urdf.xacro (robot description, xacro)
@@ -1,241 +1,152 @@
 <?xml version="1.0"?>
-<robot name="ackermann_scout" xmlns:xacro="http://ros.org/wiki/xacro">
-  <xacro:arg name="robot_namespace" default="/" />
-  <xacro:arg name="laser_enabled" default="true" />
-  <xacro:arg name="laser_xyz" default="0.1206 0.0 0.0" />
-  <xacro:arg name="laser_rpy" default="0.0 0.0 0.0" />
-  <xacro:arg name="sensor_arch_height" default="300" />
-  <xacro:include filename="$(find scout_description)/urdf/decorations.urdf.xacro" />
-  <xacro:include filename="$(find scout_description)/urdf/accessories/ydlidar_mount.urdf.xacro" />
-  <xacro:include filename="$(find scout_description)/urdf/accessories/sensor_arch.urdf.xacro" />
-  <xacro:include filename="$(find scout_description)/urdf/accessories/vlp16_mount.urdf.xacro" />
-  <xacro:property name="M_PI" value="3.14159"/>
-  <xacro:property name="base_x_size" value="0.9250000" />
-  <xacro:property name="base_y_size" value="0.380000" />
-  <xacro:property name="base_z_size" value="0.210000" />
-  <xacro:property name="wheelbase" value="0.498" />
-  <xacro:property name="track" value="0.58306" />
-  <xacro:property name="wheel_vertical_offset" value="-0.0702" />
-  <xacro:property name="wheel_length" value="1.1653e-01" />
-  <xacro:property name="wheel_radius" value="1.6459e-01" />
-  <xacro:property name="wheel_joint_friction" value="20.0" />
-  <xacro:macro name="ackermann_wheel_link" params="wheel_prefix is_right">
-    <link name="${wheel_prefix}_wheel_link">
+<robot name="agribot_ackermann_sim" xmlns:xacro="http://www.ros.org/wiki/xacro">
+  <!-- Values below are the measured physical Ackermann vehicle geometry. -->
+  <xacro:property name="wheel_radius" value="0.1275"/>
+  <xacro:property name="wheel_width" value="0.081431"/>
+  <xacro:property name="max_steering_angle" value="0.384"/>
+  <material name="sensor_black"><color rgba="0.035 0.035 0.035 1"/></material>
+  <material name="antenna_white"><color rgba="0.88 0.88 0.84 1"/></material>
+  <link name="base_link">
+    <inertial>
+      <origin xyz="0.2623915 0 0.0615505" rpy="0 0 0"/>
+      <mass value="50.0"/>
+      <inertia ixx="1.914" ixy="0" ixz="0" iyy="2.672" iyz="0" izz="4.084"/>
+    </inertial>
+    <visual name="step_vehicle_body">
+      <origin xyz="0.2794632 0.1918975 -0.7587717" rpy="0 0 1.5707963267948966"/>
+      <geometry>
+        <mesh filename="package://agribot_hardware_bringup/meshes/ackermann_vehicle_body.glb"/>
+      </geometry>
+    </visual>
+    <collision>
+      <origin xyz="0.2623915 0 0.0615505" rpy="0 0 0"/>
+      <geometry><box size="0.761611 0.631783 0.245800"/></geometry>
+    </collision>
+  </link>
+  <link name="imu_link">
+    <visual>
+      <geometry>
+        <mesh filename="package://agribot_hardware_bringup/meshes/hipnuc_n300pro.glb"/>
+      </geometry>
+    </visual>
+  </link>
+  <joint name="imu_joint" type="fixed">
+    <origin xyz="0.1425 0 0.143" rpy="0.000572424 -0.009139547 -0.000002616"/>
+    <parent link="base_link"/>
+    <child link="imu_link"/>
+  </joint>
+  <link name="lidar_link">
+    <visual>
+      <!-- C16 STEP origin is 48.55 mm below its optical center. -->
+      <origin xyz="0 0 -0.04855" rpy="0 0 3.141592653589793"/>
+      <geometry>
+        <mesh filename="package://agribot_hardware_bringup/meshes/lslidar_c16_v4.glb"/>
+      </geometry>
+    </visual>
+  </link>
+  <joint name="lidar_joint" type="fixed">
+    <origin xyz="0.48 0 0.233" rpy="-0.007648487 -0.001835661 0.000007020"/>
+    <parent link="base_link"/>
+    <child link="lidar_link"/>
+  </joint>
+  <link name="right_camera_link">
+    <visual name="camera_body">
+      <origin xyz="-0.022 0 0" rpy="0 0 0"/>
+      <geometry><box size="0.044 0.040 0.040"/></geometry>
+      <material name="sensor_black"/>
+    </visual>
+    <visual name="camera_lens">
+      <origin xyz="0.006 0 0" rpy="0 1.5707963267948966 0"/>
+      <geometry><cylinder radius="0.014" length="0.012"/></geometry>
+      <material name="sensor_black"/>
+    </visual>
+  </link>
+  <joint name="right_camera_mount_joint" type="fixed">
+    <origin xyz="0.5755 0 0.154" rpy="0 0 0"/>
+    <parent link="base_link"/>
+    <child link="right_camera_link"/>
+  </joint>
+  <link name="right_camera_optical_frame"/>
+  <joint name="right_camera_optical_joint" type="fixed">
+    <origin xyz="0 0 0" rpy="-1.5707963267948966 0 -1.5707963267948966"/>
+    <parent link="right_camera_link"/>
+    <child link="right_camera_optical_frame"/>
+  </joint>
+  <xacro:macro name="rtk_antenna" params="name y">
+    <link name="${name}">
+      <visual name="antenna_radome">
+        <origin xyz="0 0 -0.018" rpy="0 0 0"/>
+        <geometry><cylinder radius="0.0225" length="0.036"/></geometry>
+        <material name="antenna_white"/>
+      </visual>
+      <visual name="antenna_stem">
+        <origin xyz="0 0 -0.090" rpy="0 0 0"/>
+        <geometry><cylinder radius="0.008" length="0.108"/></geometry>
+        <material name="sensor_black"/>
+      </visual>
+    </link>
+    <joint name="${name}_joint" type="fixed">
+      <origin xyz="0.1425 ${y} 0.78476" rpy="0 0 0"/>
+      <parent link="base_link"/>
+      <child link="${name}"/>
+    </joint>
+  </xacro:macro>
+  <xacro:rtk_antenna name="rtk_link" y="0.2952585"/>
+  <xacro:rtk_antenna name="rtk_secondary_link" y="-0.2952585"/>
+  <xacro:macro name="wheel_link" params="name mesh">
+    <link name="${name}_wheel_link">
       <inertial>
-        <mass value="8" />
-        <origin xyz="0 0 0" />
-        <inertia ixx="0.1171" ixy="0" ixz="0" iyy="0.1361" iyz="0" izz="0.1171" />
+        <mass value="3.0"/>
+        <inertia ixx="0.01223" ixy="0" ixz="0" iyy="0.02438" iyz="0" izz="0.01223"/>
       </inertial>
       <visual>
-        <xacro:if value="${is_right}">
-          <origin xyz="0 0 0" rpy="${M_PI} 0 0" />
-        </xacro:if>
-        <xacro:unless value="${is_right}">
-          <origin xyz="0 0 0" rpy="0 0 0" />
-        </xacro:unless>
-        <geometry>
-          <mesh filename="package://scout_description/meshes/wheel.dae" />
-        </geometry>
+        <origin xyz="0 0 0" rpy="0 0 1.5707963267948966"/>
+        <geometry><mesh filename="package://agribot_hardware_bringup/meshes/${mesh}"/></geometry>
       </visual>
       <collision>
-        <origin xyz="0 0 0" rpy="${M_PI/2} 0 0" />
-        <geometry>
-          <cylinder length="${wheel_length}" radius="${wheel_radius}" />
-        </geometry>
+        <origin xyz="0 0 0" rpy="1.5707963267948966 0 0"/>
+        <geometry><cylinder radius="${wheel_radius}" length="${wheel_width}"/></geometry>
       </collision>
     </link>
   </xacro:macro>
-  <xacro:macro name="disable_gravity" params="ref">
-    <gazebo reference="${ref}">
-      <gravity>false</gravity>
-    </gazebo>
-  </xacro:macro>
-  <link name="base_link">
-    <inertial>
-      <mass value="50" />
-      <origin xyz="0.0 0.0 0.0" />
-      <inertia ixx="2.288641" ixy="0" ixz="0" iyy="5.103976" iyz="0" izz="3.431465" />
-    </inertial>
-    <visual>
-      <origin xyz="0 0 0" rpy="0 0 0" />
-      <geometry>
-        <mesh filename="package://scout_description/meshes/base_link.dae" />
-      </geometry>
-    </visual>
-    <collision>
-      <origin xyz="0 0 0.008" rpy="0 0 0" />
-      <geometry>
-        <box size="${base_x_size} ${base_y_size} ${base_z_size}"/>
-      </geometry>
-    </collision>
-    <collision>
-      <origin xyz="0 0 ${base_z_size/6}" rpy="0 0 0" />
-      <geometry>
-        <box size="${base_x_size/6} ${base_y_size*1.65} ${base_z_size/3}"/>
-      </geometry>
-    </collision>
-  </link>
-  <link name="base_footprint"/>
-  <joint name="base_footprint_joint" type="fixed">
-    <origin xyz="0 0 ${wheel_vertical_offset - wheel_radius}" rpy="0 0 0" />
-    <parent link="base_link" />
-    <child link="base_footprint" />
-  </joint>
-  <link name="imu_link"/>
-  <joint name="imu_joint" type="fixed">
-    <origin xyz="0.19 0 0.149" rpy="0 -1.5708 3.1416" />
-    <parent link="base_link" />
-    <child link="imu_link" />
-  </joint>
-  <xacro:ackermann_wheel_link wheel_prefix="front_left" is_right="false" />
-  <xacro:ackermann_wheel_link wheel_prefix="front_right" is_right="true" />
-  <xacro:ackermann_wheel_link wheel_prefix="rear_left" is_right="false" />
-  <xacro:ackermann_wheel_link wheel_prefix="rear_right" is_right="true" />
-  <link name="front_left_steering_block_link">
-    <inertial>
-      <mass value="1" />
-      <origin xyz="0 0 0" />
-      <inertia ixx="1" ixy="0" ixz="0" iyy="1" iyz="0" izz="1" />
-    </inertial>
-    <visual>
-      <origin xyz="0 0 0" rpy="0 0 0" />
-      <geometry>
-        <cylinder radius="0.03" length="0.05" />
-      </geometry>
-      <material name="dark_grey" />
-    </visual>
-  </link>
-  <link name="front_right_steering_block_link">
-    <inertial>
-      <mass value="1" />
-      <origin xyz="0 0 0" />
-      <inertia ixx="1" ixy="0" ixz="0" iyy="1" iyz="0" izz="1" />
-    </inertial>
-    <visual>
-      <origin xyz="0 0 0" rpy="0 0 0" />
-      <geometry>
-        <cylinder radius="0.03" length="0.05" />
-      </geometry>
-      <material name="dark_grey" />
-    </visual>
+  <link name="front_left_steering_link">
+    <inertial><mass value="0.2"/><inertia ixx="0.0001" ixy="0" ixz="0" iyy="0.0001" iyz="0" izz="0.0001"/></inertial>
   </link>
   <joint name="front_left_steering_joint" type="revolute">
-    <origin xyz="${wheelbase/2} ${track/2} ${wheel_vertical_offset}" rpy="0 0 0" />
-    <parent link="base_link" />
-    <child link="front_left_steering_block_link" />
-    <axis xyz="0 0 1" />
-    <limit lower="-0.7" upper="0.7" effort="200" velocity="1.5" />
-    <dynamics damping="2.0" friction="0.0" />
+    <origin xyz="0.5258472 0.2949655 0.0015843" rpy="0 0 0"/>
+    <parent link="base_link"/><child link="front_left_steering_link"/>
+    <axis xyz="0 0 1"/>
+    <limit lower="-${max_steering_angle}" upper="${max_steering_angle}" effort="200" velocity="1.5"/>
   </joint>
+  <link name="front_right_steering_link">
+    <inertial><mass value="0.2"/><inertia ixx="0.0001" ixy="0" ixz="0" iyy="0.0001" iyz="0" izz="0.0001"/></inertial>
+  </link>
   <joint name="front_right_steering_joint" type="revolute">
-    <origin xyz="${wheelbase/2} ${-track/2} ${wheel_vertical_offset}" rpy="0 0 0" />
-    <parent link="base_link" />
-    <child link="front_right_steering_block_link" />
-    <axis xyz="0 0 1" />
-    <limit lower="-0.7" upper="0.7" effort="200" velocity="1.5" />
-    <dynamics damping="2.0" friction="0.0" />
+    <origin xyz="0.5273242 -0.2949655 0.0015843" rpy="0 0 0"/>
+    <parent link="base_link"/><child link="front_right_steering_link"/>
+    <axis xyz="0 0 1"/>
+    <limit lower="-${max_steering_angle}" upper="${max_steering_angle}" effort="200" velocity="1.5"/>
   </joint>
+  <xacro:wheel_link name="front_left" mesh="ackermann_front_left_wheel.glb"/>
+  <xacro:wheel_link name="front_right" mesh="ackermann_front_right_wheel.glb"/>
+  <xacro:wheel_link name="rear_left" mesh="ackermann_rear_left_wheel.glb"/>
+  <xacro:wheel_link name="rear_right" mesh="ackermann_rear_right_wheel.glb"/>
   <joint name="front_left_wheel_joint" type="continuous">
-    <origin xyz="0 0 0" rpy="0 0 0" />
-    <parent link="front_left_steering_block_link" />
-    <child link="front_left_wheel_link" />
-    <axis xyz="0 1 0" />
-    <dynamics damping="0.0" friction="${wheel_joint_friction}" />
+    <parent link="front_left_steering_link"/><child link="front_left_wheel_link"/>
+    <axis xyz="0 1 0"/>
   </joint>
   <joint name="front_right_wheel_joint" type="continuous">
-    <origin xyz="0 0 0" rpy="0 0 0" />
-    <parent link="front_right_steering_block_link" />
-    <child link="front_right_wheel_link" />
-    <axis xyz="0 1 0" />
-    <dynamics damping="0.0" friction="${wheel_joint_friction}" />
+    <parent link="front_right_steering_link"/><child link="front_right_wheel_link"/>
+    <axis xyz="0 1 0"/>
   </joint>
   <joint name="rear_left_wheel_joint" type="continuous">
-    <origin xyz="${-wheelbase/2} ${track/2} ${wheel_vertical_offset}" rpy="0 0 0" />
-    <parent link="base_link" />
-    <child link="rear_left_wheel_link" />
-    <axis xyz="0 1 0" />
-    <dynamics damping="0.0" friction="${wheel_joint_friction}" />
+    <origin xyz="0.0000002 0.2952585 0.0000003" rpy="0 0 0"/>
+    <parent link="base_link"/><child link="rear_left_wheel_link"/>
+    <axis xyz="0 1 0"/>
   </joint>
   <joint name="rear_right_wheel_joint" type="continuous">
-    <origin xyz="${-wheelbase/2} ${-track/2} ${wheel_vertical_offset}" rpy="0 0 0" />
-    <parent link="base_link" />
-    <child link="rear_right_wheel_link" />
-    <axis xyz="0 1 0" />
-    <dynamics damping="0.0" friction="${wheel_joint_friction}" />
+    <origin xyz="0.0000002 -0.2952585 0.0000003" rpy="0 0 0"/>
+    <parent link="base_link"/><child link="rear_right_wheel_link"/>
+    <axis xyz="0 1 0"/>
   </joint>
-  <xacro:scout_decorate />
-  <xacro:if value="$(arg laser_enabled)">
-    <xacro:ydlidar_mount prefix="base"/>
-    <xacro:ydlidar frame="base_laser" topic="scan" min_range="0.65"
-      robot_namespace="$(arg robot_namespace)"/>
-    <joint name="laser_mount_joint" type="fixed">
-      <origin xyz="$(arg laser_xyz)" rpy="$(arg laser_rpy)" />
-      <parent link="top_plate_link" />
-      <child link="base_laser_mount" />
-    </joint>
-  </xacro:if>
-  <xacro:sensor_arch prefix="" parent="top_plate_link" size="$(arg sensor_arch_height)">
-    <origin xyz="0 0 0" rpy="0 0 0"/>
-  </xacro:sensor_arch>
-  <xacro:vlp16_mount
-    prefix=""
-    parent_link="sensor_arch_mount_link"
-    topic="/points"
-    robot_namespace="$(arg robot_namespace)"
-    update_rate="5"
-    horizontal_samples="360"
-    vertical_samples="16"
-    min_range="0.3"
-    max_range="25.0">
-    <origin xyz="0 0 0" rpy="0 0 0" />
-  </xacro:vlp16_mount>
-  <xacro:disable_gravity ref="base_link" />
-  <xacro:disable_gravity ref="front_left_steering_block_link" />
-  <xacro:disable_gravity ref="front_right_steering_block_link" />
-  <xacro:disable_gravity ref="front_left_wheel_link" />
-  <xacro:disable_gravity ref="front_right_wheel_link" />
-  <xacro:disable_gravity ref="rear_left_wheel_link" />
-  <xacro:disable_gravity ref="rear_right_wheel_link" />
-  <xacro:disable_gravity ref="top_plate_link" />
-  <xacro:disable_gravity ref="base_laser_mount" />
-  <xacro:disable_gravity ref="base_laser" />
-  <xacro:disable_gravity ref="sensor_arch_base_link" />
-  <xacro:disable_gravity ref="sensor_arch_mount_link" />
-  <xacro:disable_gravity ref="vlp16_mount_base_link" />
-  <xacro:disable_gravity ref="vlp16_mount_left_support" />
-  <xacro:disable_gravity ref="vlp16_mount_right_support" />
-  <xacro:disable_gravity ref="vlp16_base_link" />
-  <xacro:disable_gravity ref="vlp16" />
-  <gazebo reference="front_left_wheel_link">
-    <mu1>1.8</mu1>
-    <mu2>1.5</mu2>
-    <kp>1000000000.0</kp>
-    <kd>0.0</kd>
-    <minDepth>0.001</minDepth>
-    <fdir1>1 0 0</fdir1>
-  </gazebo>
-  <gazebo reference="front_right_wheel_link">
-    <mu1>1.8</mu1>
-    <mu2>1.5</mu2>
-    <kp>1000000000.0</kp>
-    <kd>0.0</kd>
-    <minDepth>0.001</minDepth>
-    <fdir1>1 0 0</fdir1>
-  </gazebo>
-  <gazebo reference="rear_left_wheel_link">
-    <mu1>1.8</mu1>
-    <mu2>1.5</mu2>
-    <kp>1000000000.0</kp>
-    <kd>0.0</kd>
-    <minDepth>0.001</minDepth>
-    <fdir1>1 0 0</fdir1>
-  </gazebo>
-  <gazebo reference="rear_right_wheel_link">
-    <mu1>1.8</mu1>
-    <mu2>1.5</mu2>
-    <kp>1000000000.0</kp>
-    <kd>0.0</kd>
-    <minDepth>0.001</minDepth>
-    <fdir1>1 0 0</fdir1>
-  </gazebo>
 </robot>
