Commit message: 加入大模型之前

File: ros2_ws/src/agribot_vehicle_description/generated/unity_car1/urdf/unity_car1.urdf.xacro (robot description, xacro)
@@ -4,9 +4,9 @@
   <link name="base_link">
     <inertial>
-      <origin xyz="0.312528043985 5.96046447754e-08 0.230182856321" rpy="0 0 0"/>
-      <mass value="50"/>
-      <inertia ixx="3.90099358559" ixy="0" ixz="0" iyy="8.18288230896" iyz="0" izz="7.67456102371"/>
+      <origin xyz="1.26617140659 0 0.15" rpy="0 0 0"/>
+      <mass value="6000"/>
+      <inertia ixx="7517.18824707" ixy="0" ixz="0" iyy="15768.3593833" iyz="0" izz="14788.8277172"/>
     </inertial>
-    <collision><origin xyz="0.312528043985 5.96046447754e-08 0.230182856321" rpy="0 0 0"/><geometry><box size="1.19782054424 0.638060092926 0.72740483284"/></geometry></collision>
+    <collision><origin xyz="1.25238674609 2.38852379999e-07 0.922406689519" rpy="0 0 0"/><geometry><box size="4.79999988057 2.55688415478 2.91491336289"/></geometry></collision>
     <visual name="vehicle_body">
       <origin xyz="0 0 0" rpy="0 0 0"/>
@@ -18,5 +18,5 @@
   </link>
   <joint name="imu_mount_joint" type="fixed">
-    <origin xyz="0.448928296566 0.00250006094575 0.337802886963" rpy="0 0 0"/>
+    <origin xyz="2.57 0 1.32060797228" rpy="0 0 0"/>
     <parent link="base_link"/><child link="imu_link"/>
   </joint>
@@ -25,5 +25,5 @@
   </link>
   <joint name="lidar_mount_joint" type="fixed">
-    <origin xyz="0.285124033689 0.00303386058658 0.572944641113" rpy="0 0 0"/>
+    <origin xyz="2.8 0 1.46963798028" rpy="0 0 0"/>
     <parent link="base_link"/><child link="lidar_link"/>
   </joint>
@@ -32,10 +32,10 @@
   </link>
   <joint name="right_camera_mount_joint" type="fixed">
-    <origin xyz="0.556828320026 0.00600005872548 0.345592498779" rpy="0 0 0"/>
+    <origin xyz="2.8253 0 1.58822498028" rpy="0 0 0"/>
     <parent link="base_link"/><child link="right_camera_link"/>
   </joint>
   <link name="right_camera_optical_frame"/>
   <joint name="right_camera_measurement_joint" type="fixed">
-    <origin xyz="1.42371675338e-07 1.69634937208e-08 0" rpy="-1.57079637051 0 -1.57079637051"/>
+    <origin xyz="0 0 0" rpy="-1.57079632679 0 -1.57079632679"/>
     <parent link="right_camera_link"/><child link="right_camera_optical_frame"/>
   </joint>
@@ -44,5 +44,5 @@
   </link>
   <joint name="rtk_master_mount_joint" type="fixed">
-    <origin xyz="0.180623948574 0.334000825882 1.05604362488" rpy="0 0 0"/>
+    <origin xyz="0.6 0.325 2.71803069037" rpy="0 0 0"/>
     <parent link="base_link"/><child link="rtk_link"/>
   </joint>
@@ -50,17 +50,17 @@
   </link>
   <joint name="rtk_secondary_mount_joint" type="fixed">
-    <origin xyz="0.18062402308 -0.316000819206 1.05604362488" rpy="0 0 0"/>
+    <origin xyz="0.6 -0.325 2.71803069037" rpy="0 0 0"/>
     <parent link="base_link"/><child link="rtk_secondary_link"/>
   </joint>
   <link name="front_left_steering_link"/>
   <joint name="front_left_steering_joint" type="revolute">
-    <origin xyz="0.702150940895 0.236928999424 -0.0503787994385" rpy="0 0 0"/>
+    <origin xyz="2.81371399801 0.949440360166 -0.198884554409" rpy="0 0 0"/>
     <parent link="base_link"/><child link="front_left_steering_link"/>
     <axis xyz="0 0 1"/>
-    <limit lower="-0.610865235329" upper="0.610865235329" effort="200" velocity="1.5"/>
+    <limit lower="-0.742035886603" upper="0.742035886603" effort="200" velocity="1.5"/>
   </joint>
   <link name="front_left_wheel_link">
     <visual><geometry><mesh filename="package://agribot_vehicle_description/generated/unity_car1/models/front_left_wheel_visual.obj"/></geometry></visual>
-    <collision><origin rpy="1.570796326795 0 0"/><geometry><cylinder radius="0.189735785127" length="0.154119640589"/></geometry></collision>
+    <collision><origin rpy="1.570796326795 0 0"/><geometry><cylinder radius="0.760324032115" length="0.617600240684"/></geometry></collision>
   </link>
   <joint name="front_left_wheel_joint" type="continuous">
@@ -71,12 +71,12 @@
   <link name="front_right_steering_link"/>
   <joint name="front_right_steering_joint" type="revolute">
-    <origin xyz="0.7021510005 -0.23692882061 -0.0503787994385" rpy="0 0 0"/>
+    <origin xyz="2.81371423686 -0.949439643608 -0.198884793262" rpy="0 0 0"/>
     <parent link="base_link"/><child link="front_right_steering_link"/>
     <axis xyz="0 0 1"/>
-    <limit lower="-0.610865235329" upper="0.610865235329" effort="200" velocity="1.5"/>
+    <limit lower="-0.742035886603" upper="0.742035886603" effort="200" velocity="1.5"/>
   </joint>
   <link name="front_right_wheel_link">
     <visual><geometry><mesh filename="package://agribot_vehicle_description/generated/unity_car1/models/front_right_wheel_visual.obj"/></geometry></visual>
-    <collision><origin rpy="1.570796326795 0 0"/><geometry><cylinder radius="0.189735725522" length="0.154119640589"/></geometry></collision>
+    <collision><origin rpy="1.570796326795 0 0"/><geometry><cylinder radius="0.760323793262" length="0.617600240684"/></geometry></collision>
   </link>
   <joint name="front_right_wheel_joint" type="continuous">
@@ -87,8 +87,8 @@
   <link name="rear_left_wheel_link">
     <visual><geometry><mesh filename="package://agribot_vehicle_description/generated/unity_car1/models/rear_left_wheel_visual.obj"/></geometry></visual>
-    <collision><origin rpy="1.570796326795 0 0"/><geometry><cylinder radius="0.239366620779" length="0.177247226238"/></geometry></collision>
+    <collision><origin rpy="1.570796326795 0 0"/><geometry><cylinder radius="0.959208586524" length="0.710278905187"/></geometry></collision>
   </link>
   <joint name="rear_left_wheel_joint" type="continuous">
-    <origin xyz="-3.99365838177e-08 0.228484243155 0" rpy="0 0 0"/>
+    <origin xyz="-1.60036992584e-07 0.915599874394 0" rpy="0 0 0"/>
     <parent link="base_link"/><child link="rear_left_wheel_link"/>
     <axis xyz="0 1 0"/>
@@ -96,8 +96,8 @@
   <link name="rear_right_wheel_link">
     <visual><geometry><mesh filename="package://agribot_vehicle_description/generated/unity_car1/models/rear_right_wheel_visual.obj"/></geometry></visual>
-    <collision><origin rpy="1.570796326795 0 0"/><geometry><cylinder radius="0.239366620779" length="0.177247315645"/></geometry></collision>
+    <collision><origin rpy="1.570796326795 0 0"/><geometry><cylinder radius="0.959208586524" length="0.710279263466"/></geometry></collision>
   </link>
   <joint name="rear_right_wheel_joint" type="continuous">
-    <origin xyz="1.45382976768e-08 -0.228484228253 0" rpy="0 0 0"/>
+    <origin xyz="5.82590000213e-08 -0.91559981468 0" rpy="0 0 0"/>
     <parent link="base_link"/><child link="rear_right_wheel_link"/>
     <axis xyz="0 1 0"/>

File: ros2_ws/src/agribot_vehicle_description/generated/unity_car2/urdf/unity_car2.urdf.xacro (robot description, xacro)
@@ -4,9 +4,9 @@
   <link name="base_link">
     <inertial>
-      <origin xyz="0.424725353718 -0.000142782926559 0.222903773189" rpy="0 0 0"/>
-      <mass value="50"/>
-      <inertia ixx="5.20898628235" ixy="0" ixz="0" iyy="11.680355072" iyz="0" izz="11.8959083557"/>
+      <origin xyz="1.24139535061 0 0.15" rpy="0 0 0"/>
+      <mass value="7000"/>
+      <inertia ixx="8946.67863643" ixy="0" ixz="0" iyy="20061.5601656" iyz="0" izz="20431.7826044"/>
     </inertial>
-    <collision><origin xyz="0.424725353718 -0.000142782926559 0.222903773189" rpy="0 0 0"/><geometry><box size="1.48461222649 0.806811451912 0.774087846279"/></geometry></collision>
+    <collision><origin xyz="1.4876421676 -0.000500111190689 0.780742306554" rpy="0 0 0"/><geometry><box size="5.19999979123 2.82593616478 2.71131852967"/></geometry></collision>
     <visual name="vehicle_body">
       <origin xyz="0 0 0" rpy="0 0 0"/>
@@ -18,5 +18,5 @@
   </link>
   <joint name="imu_mount_joint" type="fixed">
-    <origin xyz="0.195598676801 0.00038285276969 0.682819366455" rpy="0 0 0"/>
+    <origin xyz="2.47 0 1.12114728821" rpy="0 0 0"/>
     <parent link="base_link"/><child link="imu_link"/>
   </joint>
@@ -25,5 +25,5 @@
   </link>
   <joint name="lidar_mount_joint" type="fixed">
-    <origin xyz="0.508300125599 0.00498151686043 0.4319190979" rpy="0 0 0"/>
+    <origin xyz="2.7 0 1.27017729621" rpy="0 0 0"/>
     <parent link="base_link"/><child link="lidar_link"/>
   </joint>
@@ -32,10 +32,10 @@
   </link>
   <joint name="right_camera_mount_joint" type="fixed">
-    <origin xyz="0.628299117088 0.00204264582135 0.407718658447" rpy="0 0 0"/>
+    <origin xyz="2.7253 0 1.38876429621" rpy="0 0 0"/>
     <parent link="base_link"/><child link="right_camera_link"/>
   </joint>
   <link name="right_camera_optical_frame"/>
   <joint name="right_camera_measurement_joint" type="fixed">
-    <origin xyz="-4.0350453645e-08 1.13871514884e-07 0" rpy="-1.57079637051 0 -1.57079637051"/>
+    <origin xyz="0 0 0" rpy="-1.57079632679 0 -1.57079632679"/>
     <parent link="right_camera_link"/><child link="right_camera_optical_frame"/>
   </joint>
@@ -44,5 +44,5 @@
   </link>
   <joint name="rtk_master_mount_joint" type="fixed">
-    <origin xyz="0.0951080694795 0.338216036558 1.19421768188" rpy="0 0 0"/>
+    <origin xyz="0.6 0.325 2.71425545582" rpy="0 0 0"/>
     <parent link="base_link"/><child link="rtk_link"/>
   </joint>
@@ -50,17 +50,17 @@
   </link>
   <joint name="rtk_secondary_mount_joint" type="fixed">
-    <origin xyz="0.0948976054788 -0.311785399914 1.19421768188" rpy="0 0 0"/>
+    <origin xyz="0.6 -0.325 2.71425545582" rpy="0 0 0"/>
     <parent link="base_link"/><child link="rtk_secondary_link"/>
   </joint>
   <link name="front_left_steering_link"/>
   <joint name="front_left_steering_joint" type="revolute">
-    <origin xyz="0.787711083889 0.333970189095 -0.0740814208984" rpy="0 0 0"/>
+    <origin xyz="2.75903525425 1.16976331097 -0.196197242286" rpy="0 0 0"/>
     <parent link="base_link"/><child link="front_left_steering_link"/>
     <axis xyz="0 0 1"/>
-    <limit lower="-0.610865235329" upper="0.610865235329" effort="200" velocity="1.5"/>
+    <limit lower="-0.783345204608" upper="0.783345204608" effort="200" velocity="1.5"/>
   </joint>
   <link name="front_left_wheel_link">
     <visual><geometry><mesh filename="package://agribot_vehicle_description/generated/unity_car2/models/front_left_wheel_visual.obj"/></geometry></visual>
-    <collision><origin rpy="1.570796326795 0 0"/><geometry><cylinder radius="0.213691115379" length="0.168684005737"/></geometry></collision>
+    <collision><origin rpy="1.570796326795 0 0"/><geometry><cylinder radius="0.748474069886" length="0.590832258396"/></geometry></collision>
   </link>
   <joint name="front_left_wheel_joint" type="continuous">
@@ -71,12 +71,12 @@
   <link name="front_right_steering_link"/>
   <joint name="front_right_steering_joint" type="revolute">
-    <origin xyz="0.787494540215 -0.333970040083 -0.0740814208984" rpy="0 0 0"/>
+    <origin xyz="2.75827678882 -1.16976278905 -0.196605494189" rpy="0 0 0"/>
     <parent link="base_link"/><child link="front_right_steering_link"/>
     <axis xyz="0 0 1"/>
-    <limit lower="-0.610865235329" upper="0.610865235329" effort="200" velocity="1.5"/>
+    <limit lower="-0.783345204608" upper="0.783345204608" effort="200" velocity="1.5"/>
   </joint>
   <link name="front_right_wheel_link">
     <visual><geometry><mesh filename="package://agribot_vehicle_description/generated/unity_car2/models/front_right_wheel_visual.obj"/></geometry></visual>
-    <collision><origin rpy="1.570796326795 0 0"/><geometry><cylinder radius="0.213574558496" length="0.168683886528"/></geometry></collision>
+    <collision><origin rpy="1.570796326795 0 0"/><geometry><cylinder radius="0.748065817983" length="0.590831840854"/></geometry></collision>
   </link>
   <joint name="front_right_wheel_joint" type="continuous">
@@ -87,8 +87,8 @@
   <link name="rear_left_wheel_link">
     <visual><geometry><mesh filename="package://agribot_vehicle_description/generated/unity_car2/models/rear_left_wheel_visual.obj"/></geometry></visual>
-    <collision><origin rpy="1.570796326795 0 0"/><geometry><cylinder radius="0.269663333893" length="0.229978859425"/></geometry></collision>
+    <collision><origin rpy="1.570796326795 0 0"/><geometry><cylinder radius="0.9445222496" length="0.805523489339"/></geometry></collision>
   </link>
   <joint name="rear_left_wheel_joint" type="continuous">
-    <origin xyz="5.99944796704e-05 0.291460156441 -9.53674316406e-06" rpy="0 0 0"/>
+    <origin xyz="0.000210136543533 1.02086775631 -0.000149062571552" rpy="0 0 0"/>
     <parent link="base_link"/><child link="rear_left_wheel_link"/>
     <axis xyz="0 1 0"/>
@@ -96,8 +96,8 @@
   <link name="rear_right_wheel_link">
     <visual><geometry><mesh filename="package://agribot_vehicle_description/generated/unity_car2/models/rear_right_wheel_visual.obj"/></geometry></visual>
-    <collision><origin rpy="1.570796326795 0 0"/><geometry><cylinder radius="0.269748449326" length="0.229978859425"/></geometry></collision>
+    <collision><origin rpy="1.570796326795 0 0"/><geometry><cylinder radius="0.944820374743" length="0.805523489339"/></geometry></collision>
   </link>
   <joint name="rear_right_wheel_joint" type="continuous">
-    <origin xyz="-6.01439896855e-05 -0.291460156441 9.53674316406e-06" rpy="0 0 0"/>
+    <origin xyz="-0.000210660217011 -1.02086775631 0.000149062571552" rpy="0 0 0"/>
     <parent link="base_link"/><child link="rear_right_wheel_link"/>
     <axis xyz="0 1 0"/>
