Commit message: 加入大模型之前

File: ros2_ws/src/agribot_vehicle_description/generated/unity_car3/urdf/unity_car3.urdf.xacro (robot description, xacro)
@@ -85,10 +85,10 @@
       <origin rpy="1.570796326795 0 0" />
       <geometry>
-        <cylinder radius="0.224918439984" length="0.154119610786" />
+        <cylinder radius="0.118148150498" length="0.15" />
       </geometry>
     </collision>
   </link>
   <joint name="front_left_wheel_joint" type="continuous">
-    <origin xyz="0.200999945402 0.294500052929 0" rpy="0 0 0" />
+    <origin xyz="0.448938366814 0.303675957024 -0.106944138711" rpy="0 0 0" />
     <parent link="base_link" />
     <child link="front_left_wheel_link" />
@@ -99,10 +99,10 @@
       <origin rpy="1.570796326795 0 0" />
       <geometry>
-        <cylinder radius="0.224918439984" length="0.154119729996" />
+        <cylinder radius="0.118148146635" length="0.15" />
       </geometry>
     </collision>
   </link>
   <joint name="front_right_wheel_joint" type="continuous">
-    <origin xyz="0.201000019908 -0.294500023127 0" rpy="0 0 0" />
+    <origin xyz="0.448938430263 -0.297507204115 -0.10694420218" rpy="0 0 0" />
     <parent link="base_link" />
     <child link="front_right_wheel_link" />
@@ -113,10 +113,10 @@
       <origin rpy="1.570796326795 0 0" />
       <geometry>
-        <cylinder radius="0.224918439984" length="0.154119610786" />
+        <cylinder radius="0.118148150498" length="0.15" />
       </geometry>
     </collision>
   </link>
   <joint name="rear_left_wheel_joint" type="continuous">
-    <origin xyz="-0.201000079513 0.294499993324 0" rpy="0 0 0" />
+    <origin xyz="-0.388064739151 0.303675957024 -0.106944138711" rpy="0 0 0" />
     <parent link="base_link" />
     <child link="rear_left_wheel_link" />
@@ -127,10 +127,10 @@
       <origin rpy="1.570796326795 0 0" />
       <geometry>
-        <cylinder radius="0.224918439984" length="0.154119610786" />
+        <cylinder radius="0.118148146635" length="0.15" />
       </geometry>
     </collision>
   </link>
   <joint name="rear_right_wheel_joint" type="continuous">
-    <origin xyz="-0.201000005007 -0.294500052929 0" rpy="0 0 0" />
+    <origin xyz="-0.388064683391 -0.297507204115 -0.10694420218" rpy="0 0 0" />
     <parent link="base_link" />
     <child link="rear_right_wheel_link" />
@@ -319,3 +319,199 @@
     <limit lower="0" upper="0.0089" effort="5" velocity="0.05" />
   </joint>
+  <link name="display_left_sprocket_link">
+    <visual>
+      <geometry>
+        <mesh filename="package://agribot_vehicle_description/generated/unity_car3/models/rotor_left_sprocket.obj" />
+      </geometry>
+    </visual>
+  </link>
+  <joint name="display_left_sprocket_joint" type="continuous">
+    <parent link="base_link" />
+    <child link="display_left_sprocket_link" />
+    <origin xyz="0.035841906608619245 0.30700362980921403 0.07214649872863443" rpy="0 0 0" />
+    <axis xyz="0 1 0" />
+    <mimic joint="front_left_wheel_joint" multiplier="0.9313421109302513" offset="0" />
+  </joint>
+  <link name="display_left_idler_front_link">
+    <visual>
+      <geometry>
+        <mesh filename="package://agribot_vehicle_description/generated/unity_car3/models/rotor_left_idler_front.obj" />
+      </geometry>
+    </visual>
+  </link>
+  <joint name="display_left_idler_front_joint" type="continuous">
+    <parent link="base_link" />
+    <child link="display_left_idler_front_link" />
+    <origin xyz="0.44893836681393606 0.30367595702409744 -0.10694413871123133" rpy="0 0 0" />
+    <axis xyz="0 1 0" />
+    <mimic joint="front_left_wheel_joint" multiplier="1.3621552730685873" offset="0" />
+  </joint>
+  <link name="display_left_idler_back_link">
+    <visual>
+      <geometry>
+        <mesh filename="package://agribot_vehicle_description/generated/unity_car3/models/rotor_left_idler_back.obj" />
+      </geometry>
+    </visual>
+  </link>
+  <joint name="display_left_idler_back_joint" type="continuous">
+    <parent link="base_link" />
+    <child link="display_left_idler_back_link" />
+    <origin xyz="-0.38806473915127737 0.30367595702409744 -0.10694413871123133" rpy="0 0 0" />
+    <axis xyz="0 1 0" />
+    <mimic joint="rear_left_wheel_joint" multiplier="1.3621552730685873" offset="0" />
+  </joint>
+  <link name="display_left_roller_0_link">
+    <visual>
+      <geometry>
+        <mesh filename="package://agribot_vehicle_description/generated/unity_car3/models/rotor_left_roller_0.obj" />
+      </geometry>
+    </visual>
+  </link>
+  <joint name="display_left_roller_0_joint" type="continuous">
+    <parent link="base_link" />
+    <child link="display_left_roller_0_link" />
+    <origin xyz="0.2471377092406679 0.30341892689466476 -0.14649352829701656" rpy="0 0 0" />
+    <axis xyz="0 1 0" />
+    <mimic joint="front_left_wheel_joint" multiplier="2.4180767559931597" offset="0" />
+  </joint>
+  <link name="display_left_roller_1_link">
+    <visual>
+      <geometry>
+        <mesh filename="package://agribot_vehicle_description/generated/unity_car3/models/rotor_left_roller_1.obj" />
+      </geometry>
+    </visual>
+  </link>
+  <joint name="display_left_roller_1_joint" type="continuous">
+    <parent link="base_link" />
+    <child link="display_left_roller_1_link" />
+    <origin xyz="0.1008230393319573 0.30341892689466476 -0.14649221159590836" rpy="0 0 0" />
+    <axis xyz="0 1 0" />
+    <mimic joint="front_left_wheel_joint" multiplier="2.4180751998650827" offset="0" />
+  </joint>
+  <link name="display_left_roller_2_link">
+    <visual>
+      <geometry>
+        <mesh filename="package://agribot_vehicle_description/generated/unity_car3/models/rotor_left_roller_2.obj" />
+      </geometry>
+    </visual>
+  </link>
+  <joint name="display_left_roller_2_joint" type="continuous">
+    <parent link="base_link" />
+    <child link="display_left_roller_2_link" />
+    <origin xyz="-0.040638400140649455 0.30341892689466476 -0.14649352829701656" rpy="0 0 0" />
+    <axis xyz="0 1 0" />
+    <mimic joint="front_left_wheel_joint" multiplier="2.4180751998650827" offset="0" />
+  </joint>
+  <link name="display_left_roller_3_link">
+    <visual>
+      <geometry>
+        <mesh filename="package://agribot_vehicle_description/generated/unity_car3/models/rotor_left_roller_3.obj" />
+      </geometry>
+    </visual>
+  </link>
+  <joint name="display_left_roller_3_joint" type="continuous">
+    <parent link="base_link" />
+    <child link="display_left_roller_3_link" />
+    <origin xyz="-0.18583391754294554 0.30341892689466476 -0.14649221159590836" rpy="0 0 0" />
+    <axis xyz="0 1 0" />
+    <mimic joint="front_left_wheel_joint" multiplier="2.4522298978990795" offset="0" />
+  </joint>
+  <link name="display_right_sprocket_link">
+    <visual>
+      <geometry>
+        <mesh filename="package://agribot_vehicle_description/generated/unity_car3/models/rotor_right_sprocket.obj" />
+      </geometry>
+    </visual>
+  </link>
+  <joint name="display_right_sprocket_joint" type="continuous">
+    <parent link="base_link" />
+    <child link="display_right_sprocket_link" />
+    <origin xyz="0.02503175821408432 -0.3059225191757157 0.07214642939517252" rpy="0 0 0" />
+    <axis xyz="0 1 0" />
+    <mimic joint="front_right_wheel_joint" multiplier="0.9313419955517421" offset="0" />
+  </joint>
+  <link name="display_right_idler_back_link">
+    <visual>
+      <geometry>
+        <mesh filename="package://agribot_vehicle_description/generated/unity_car3/models/rotor_right_idler_back.obj" />
+      </geometry>
+    </visual>
+  </link>
+  <joint name="display_right_idler_back_joint" type="continuous">
+    <parent link="base_link" />
+    <child link="display_right_idler_back_link" />
+    <origin xyz="-0.3880646833907003 -0.2975072041153908 -0.10694420217950963" rpy="0 0 0" />
+    <axis xyz="0 1 0" />
+    <mimic joint="rear_right_wheel_joint" multiplier="1.3621552731342519" offset="0" />
+  </joint>
+  <link name="display_right_idler_front_link">
+    <visual>
+      <geometry>
+        <mesh filename="package://agribot_vehicle_description/generated/unity_car3/models/rotor_right_idler_front.obj" />
+      </geometry>
+    </visual>
+  </link>
+  <joint name="display_right_idler_front_joint" type="continuous">
+    <parent link="base_link" />
+    <child link="display_right_idler_front_link" />
+    <origin xyz="0.44893843026264857 -0.2975072041153908 -0.10694420217950963" rpy="0 0 0" />
+    <axis xyz="0 1 0" />
+    <mimic joint="front_right_wheel_joint" multiplier="1.3621552731342519" offset="0" />
+  </joint>
+  <link name="display_right_roller_0_link">
+    <visual>
+      <geometry>
+        <mesh filename="package://agribot_vehicle_description/generated/unity_car3/models/rotor_right_roller_0.obj" />
+      </geometry>
+    </visual>
+  </link>
+  <joint name="display_right_roller_0_joint" type="continuous">
+    <parent link="base_link" />
+    <child link="display_right_roller_0_link" />
+    <origin xyz="-0.1862639895279778 -0.29658111184835434 -0.14649359047006005" rpy="0 0 0" />
+    <axis xyz="0 1 0" />
+    <mimic joint="front_right_wheel_joint" multiplier="2.418075199981649" offset="0" />
+  </joint>
+  <link name="display_right_roller_1_link">
+    <visual>
+      <geometry>
+        <mesh filename="package://agribot_vehicle_description/generated/unity_car3/models/rotor_right_roller_1.obj" />
+      </geometry>
+    </visual>
+  </link>
+  <joint name="display_right_roller_1_joint" type="continuous">
+    <parent link="base_link" />
+    <child link="display_right_roller_1_link" />
+    <origin xyz="-0.04831964638873276 -0.29658111184835434 -0.14649227376899496" rpy="0 0 0" />
+    <axis xyz="0 1 0" />
+    <mimic joint="front_right_wheel_joint" multiplier="2.452229898017292" offset="0" />
+  </joint>
+  <link name="display_right_roller_2_link">
+    <visual>
+      <geometry>
+        <mesh filename="package://agribot_vehicle_description/generated/unity_car3/models/rotor_right_roller_2.obj" />
+      </geometry>
+    </visual>
+  </link>
+  <joint name="display_right_roller_2_joint" type="continuous">
+    <parent link="base_link" />
+    <child link="display_right_roller_2_link" />
+    <origin xyz="0.10151201614371613 -0.29658111184835434 -0.14649359047006005" rpy="0 0 0" />
+    <axis xyz="0 1 0" />
+    <mimic joint="front_right_wheel_joint" multiplier="2.4180759780454375" offset="0" />
+  </joint>
+  <link name="display_right_roller_3_link">
+    <visual>
+      <geometry>
+        <mesh filename="package://agribot_vehicle_description/generated/unity_car3/models/rotor_right_roller_3.obj" />
+      </geometry>
+    </visual>
+  </link>
+  <joint name="display_right_roller_3_joint" type="continuous">
+    <parent link="base_link" />
+    <child link="display_right_roller_3_link" />
+    <origin xyz="0.2405754209870814 -0.29658111184835434 -0.14649227376899496" rpy="0 0 0" />
+    <axis xyz="0 1 0" />
+    <mimic joint="front_right_wheel_joint" multiplier="2.4180767561097265" offset="0" />
+  </joint>
 </robot>

File: ros2_ws/src/agribot_vehicle_description/generated/unity_car4/urdf/unity_car4.urdf.xacro (robot description, xacro)
@@ -4,9 +4,9 @@
   <link name="base_link">
     <inertial>
-      <origin xyz="0.263963907957 -4.74750995636e-05 0.237996518612" rpy="0 0 0"/>
-      <mass value="50"/>
-      <inertia ixx="3.74930953979" ixy="0" ixz="0" iyy="8.11046791077" iyz="0" izz="7.62208414078"/>
+      <origin xyz="0.983305886074 0 0.15" rpy="0 0 0"/>
+      <mass value="2500"/>
+      <inertia ixx="1689.54889862" ixy="0" ixz="0" iyy="3654.81444006" iyz="0" izz="3434.73445856"/>
     </inertial>
-    <collision><origin xyz="0.263963907957 -4.74750995636e-05 0.237996518612" rpy="0 0 0"/><geometry><box size="1.19916188717 0.625548601151 0.713108181953"/></geometry></collision>
+    <collision><origin xyz="0.792445141963 -0.000142551923975 0.714486632087" rpy="0 0 0"/><geometry><box size="3.6 1.87795777404 2.14081977576"/></geometry></collision>
     <visual name="vehicle_body">
       <origin xyz="0 0 0" rpy="0 0 0"/>
@@ -18,5 +18,5 @@
   </link>
   <joint name="imu_mount_joint" type="fixed">
-    <origin xyz="0.353028059006 0.00789905898273 0.294473648071" rpy="0 0 0"/>
+    <origin xyz="1.72 0 0.920368656051" rpy="0 0 0"/>
     <parent link="base_link"/><child link="imu_link"/>
   </joint>
@@ -25,5 +25,5 @@
   </link>
   <joint name="lidar_mount_joint" type="fixed">
-    <origin xyz="0.633336246014 0.000815762614366 0.41477394104" rpy="0 0 0"/>
+    <origin xyz="1.95 0 1.35939866405" rpy="0 0 0"/>
     <parent link="base_link"/><child link="lidar_link"/>
   </joint>
@@ -32,10 +32,10 @@
   </link>
   <joint name="right_camera_mount_joint" type="fixed">
-    <origin xyz="0.658633291721 0.0034443042241 0.517072677612" rpy="0 0 0"/>
+    <origin xyz="1.9753 0 1.47798566405" rpy="0 0 0"/>
     <parent link="base_link"/><child link="right_camera_link"/>
   </joint>
   <link name="right_camera_optical_frame"/>
   <joint name="right_camera_measurement_joint" type="fixed">
-    <origin xyz="3.19319255482e-08 1.09499460166e-07 0" rpy="-1.57079637051 0 -1.57079637051"/>
+    <origin xyz="0 0 0" rpy="-1.57079632679 0 -1.57079632679"/>
     <parent link="right_camera_link"/><child link="right_camera_optical_frame"/>
   </joint>
@@ -44,5 +44,5 @@
   </link>
   <joint name="rtk_master_mount_joint" type="fixed">
-    <origin xyz="0.522781550884 0.314591765404 0.807771682739" rpy="0 0 0"/>
+    <origin xyz="1.6 0.325 1.44550812546" rpy="0 0 0"/>
     <parent link="base_link"/><child link="rtk_link"/>
   </joint>
@@ -50,17 +50,17 @@
   </link>
   <joint name="rtk_secondary_mount_joint" type="fixed">
-    <origin xyz="0.523516178131 -0.335409253836 0.807771682739" rpy="0 0 0"/>
+    <origin xyz="1.6 -0.325 1.44550812546" rpy="0 0 0"/>
     <parent link="base_link"/><child link="rtk_secondary_link"/>
   </joint>
   <link name="front_left_steering_link"/>
   <joint name="front_left_steering_joint" type="revolute">
-    <origin xyz="0.727570712566 0.261286228895 -0.106220245361" rpy="0 0 0"/>
+    <origin xyz="2.18423784074 0.784406377413 -0.313106738531" rpy="0 0 0"/>
     <parent link="base_link"/><child link="front_left_steering_link"/>
     <axis xyz="0 0 1"/>
-    <limit lower="-0.610865235329" upper="0.610865235329" effort="200" velocity="1.5"/>
+    <limit lower="-0.751980612199" upper="0.751980612199" effort="200" velocity="1.5"/>
   </joint>
   <link name="front_left_wheel_link">
     <visual><geometry><mesh filename="package://agribot_vehicle_description/generated/unity_car4/models/front_left_wheel_visual.obj"/></geometry></visual>
-    <collision><origin rpy="1.570796326795 0 0"/><geometry><cylinder radius="0.134206175804" length="0.0503803491592"/></geometry></collision>
+    <collision><origin rpy="1.570796326795 0 0"/><geometry><cylinder radius="0.402899934555" length="0.151246320345"/></geometry></collision>
   </link>
   <joint name="front_left_wheel_joint" type="continuous">
@@ -71,12 +71,12 @@
   <link name="front_right_steering_link"/>
   <joint name="front_right_steering_joint" type="revolute">
-    <origin xyz="0.728161156178 -0.261286020279 -0.106220245361" rpy="0 0 0"/>
+    <origin xyz="2.18601040802 -0.784406109835 -0.3132023306" rpy="0 0 0"/>
     <parent link="base_link"/><child link="front_right_steering_link"/>
     <axis xyz="0 0 1"/>
-    <limit lower="-0.610865235329" upper="0.610865235329" effort="200" velocity="1.5"/>
+    <limit lower="-0.751980612199" upper="0.751980612199" effort="200" velocity="1.5"/>
   </joint>
   <link name="front_right_wheel_link">
     <visual><geometry><mesh filename="package://agribot_vehicle_description/generated/unity_car4/models/front_right_wheel_visual.obj"/></geometry></visual>
-    <collision><origin rpy="1.570796326795 0 0"/><geometry><cylinder radius="0.134174332023" length="0.0503802895546"/></geometry></collision>
+    <collision><origin rpy="1.570796326795 0 0"/><geometry><cylinder radius="0.402804342486" length="0.151246320345"/></geometry></collision>
   </link>
   <joint name="front_right_wheel_joint" type="continuous">
@@ -87,8 +87,8 @@
   <link name="rear_left_wheel_link">
     <visual><geometry><mesh filename="package://agribot_vehicle_description/generated/unity_car4/models/rear_left_wheel_visual.obj"/></geometry></visual>
-    <collision><origin rpy="1.570796326795 0 0"/><geometry><cylinder radius="0.238504588604" length="0.108189404011"/></geometry></collision>
+    <collision><origin rpy="1.570796326795 0 0"/><geometry><cylinder radius="0.716013964573" length="0.324794959434"/></geometry></collision>
   </link>
   <joint name="rear_left_wheel_joint" type="continuous">
-    <origin xyz="-0.000335376040312 0.297314196825 -1.90734863281e-06" rpy="0 0 0"/>
+    <origin xyz="-0.00100688748051 0.89256602754 7.29148742995e-06" rpy="0 0 0"/>
     <parent link="base_link"/><child link="rear_left_wheel_link"/>
     <axis xyz="0 1 0"/>
@@ -96,8 +96,8 @@
   <link name="rear_right_wheel_link">
     <visual><geometry><mesh filename="package://agribot_vehicle_description/generated/unity_car4/models/rear_right_wheel_visual.obj"/></geometry></visual>
-    <collision><origin rpy="1.570796326795 0 0"/><geometry><cylinder radius="0.238499730825" length="0.108189463615"/></geometry></collision>
+    <collision><origin rpy="1.570796326795 0 0"/><geometry><cylinder radius="0.715999381599" length="0.324795227012"/></geometry></collision>
   </link>
   <joint name="rear_right_wheel_joint" type="continuous">
-    <origin xyz="0.000335412711138 -0.297313958406 3.81469726562e-06" rpy="0 0 0"/>
+    <origin xyz="0.0010068736966 -0.89256555928 -7.29148743006e-06" rpy="0 0 0"/>
     <parent link="base_link"/><child link="rear_right_wheel_link"/>
     <axis xyz="0 1 0"/>
