Commit message: 加入大模型之前

File: ros2_ws/src/agribot_vehicle_description/generated/unity_car5/urdf/unity_car5.urdf.xacro (robot description, xacro)
@@ -4,9 +4,9 @@
   <link name="base_link">
     <inertial>
-      <origin xyz="0.297903060913 0.0118678212166 0.339076757431" rpy="0 0 0"/>
-      <mass value="50"/>
-      <inertia ixx="4.88102436066" ixy="0" ixz="0" iyy="10.9684906006" iyz="0" izz="9.20778274536"/>
+      <origin xyz="0.749556315148 0 0.15" rpy="0 0 0"/>
+      <mass value="1400"/>
+      <inertia ixx="860.773734831" ixy="0" ixz="0" iyy="1934.30491427" iyz="0" izz="1623.80215389"/>
     </inertial>
-    <collision><origin xyz="0.297903060913 0.0118678212166 0.339076757431" rpy="0 0 0"/><geometry><box size="1.35478043556 0.611913323402 0.892753005028"/></geometry></collision>
+    <collision><origin xyz="0.747626981109 0.0297838609691 0.850957797296" rpy="0 0 0"/><geometry><box size="3.4 1.53567710675 2.24048128938"/></geometry></collision>
     <visual name="vehicle_body">
       <origin xyz="0 0 0" rpy="0 0 0"/>
@@ -18,5 +18,5 @@
   </link>
   <joint name="imu_mount_joint" type="fixed">
-    <origin xyz="0.441098928452 -0.000132109504193 0.201900482178" rpy="0 0 0"/>
+    <origin xyz="1.37 0 0.5468719553" rpy="0 0 0"/>
     <parent link="base_link"/><child link="imu_link"/>
   </joint>
@@ -25,5 +25,5 @@
   </link>
   <joint name="lidar_mount_joint" type="fixed">
-    <origin xyz="0.577098965645 -0.00013209329336 0.2327003479" rpy="0 0 0"/>
+    <origin xyz="1.6 0 0.6959019633" rpy="0 0 0"/>
     <parent link="base_link"/><child link="lidar_link"/>
   </joint>
@@ -32,10 +32,10 @@
   </link>
   <joint name="right_camera_mount_joint" type="fixed">
-    <origin xyz="0.60239893198 0.00246786465868 0.214900970459" rpy="0 0 0"/>
+    <origin xyz="1.6253 0 0.8144889633" rpy="0 0 0"/>
     <parent link="base_link"/><child link="right_camera_link"/>
   </joint>
   <link name="right_camera_optical_frame"/>
   <joint name="right_camera_measurement_joint" type="fixed">
-    <origin xyz="1.1919689058e-07 -6.06825523164e-09 0" rpy="-1.57079637051 0 -1.57079637051"/>
+    <origin xyz="0 0 0" rpy="-1.57079632679 0 -1.57079632679"/>
     <parent link="right_camera_link"/><child link="right_camera_optical_frame"/>
   </joint>
@@ -44,5 +44,5 @@
   </link>
   <joint name="rtk_master_mount_joint" type="fixed">
-    <origin xyz="0.36309877038 0.324868559837 0.71190071106" rpy="0 0 0"/>
+    <origin xyz="1.1 0.325 1.0600262053" rpy="0 0 0"/>
     <parent link="base_link"/><child link="rtk_link"/>
   </joint>
@@ -50,17 +50,17 @@
   </link>
   <joint name="rtk_secondary_mount_joint" type="fixed">
-    <origin xyz="0.363098919392 -0.325132846832 0.71190071106" rpy="0 0 0"/>
+    <origin xyz="1.1 -0.325 1.0600262053" rpy="0 0 0"/>
     <parent link="base_link"/><child link="rtk_secondary_link"/>
   </joint>
   <link name="front_left_steering_link"/>
   <joint name="front_left_steering_joint" type="revolute">
-    <origin xyz="0.66371512413 0.242358237505 -0.0844879150391" rpy="0 0 0"/>
+    <origin xyz="1.66568055074 0.608229928546 -0.171873288014" rpy="0 0 0"/>
     <parent link="base_link"/><child link="front_left_steering_link"/>
     <axis xyz="0 0 1"/>
-    <limit lower="-0.610865235329" upper="0.610865235329" effort="200" velocity="1.5"/>
+    <limit lower="-0.754872334327" upper="0.754872334327" effort="200" velocity="1.5"/>
   </joint>
   <link name="front_left_wheel_link">
     <visual><geometry><mesh filename="package://agribot_vehicle_description/generated/unity_car5/models/front_left_wheel_visual.obj"/></geometry></visual>
-    <collision><origin rpy="1.570796326795 0 0"/><geometry><cylinder radius="0.102811448276" length="0.0696836709976"/></geometry></collision>
+    <collision><origin rpy="1.570796326795 0 0"/><geometry><cylinder radius="0.258018875209" length="0.174880353431"/></geometry></collision>
   </link>
   <joint name="front_left_wheel_joint" type="continuous">
@@ -71,12 +71,12 @@
   <link name="front_right_steering_link"/>
   <joint name="front_right_steering_joint" type="revolute">
-    <origin xyz="0.663715183735 -0.242358058691 -0.0844879150391" rpy="0 0 0"/>
+    <origin xyz="1.66568070033 -0.608229479788 -0.171873269315" rpy="0 0 0"/>
     <parent link="base_link"/><child link="front_right_steering_link"/>
     <axis xyz="0 0 1"/>
-    <limit lower="-0.610865235329" upper="0.610865235329" effort="200" velocity="1.5"/>
+    <limit lower="-0.754872334327" upper="0.754872334327" effort="200" velocity="1.5"/>
   </joint>
   <link name="front_right_wheel_link">
     <visual><geometry><mesh filename="package://agribot_vehicle_description/generated/unity_car5/models/front_right_wheel_visual.obj"/></geometry></visual>
-    <collision><origin rpy="1.570796326795 0 0"/><geometry><cylinder radius="0.102811455727" length="0.0696836709976"/></geometry></collision>
+    <collision><origin rpy="1.570796326795 0 0"/><geometry><cylinder radius="0.258018893907" length="0.174880353431"/></geometry></collision>
   </link>
   <joint name="front_right_wheel_joint" type="continuous">
@@ -87,8 +87,8 @@
   <link name="rear_left_wheel_link">
     <visual><geometry><mesh filename="package://agribot_vehicle_description/generated/unity_car5/models/rear_left_wheel_visual.obj"/></geometry></visual>
-    <collision><origin rpy="1.570796326795 0 0"/><geometry><cylinder radius="0.171295493841" length="0.162000030279"/></geometry></collision>
+    <collision><origin rpy="1.570796326795 0 0"/><geometry><cylinder radius="0.429888610562" length="0.406560420044"/></geometry></collision>
   </link>
   <joint name="rear_left_wheel_joint" type="continuous">
-    <origin xyz="-3.61019729667e-08 0.202810227871 0" rpy="0 0 0"/>
+    <origin xyz="-9.06026577183e-08 0.508978987783 -3.55266059299e-06" rpy="0 0 0"/>
     <parent link="base_link"/><child link="rear_left_wheel_link"/>
     <axis xyz="0 1 0"/>
@@ -96,8 +96,8 @@
   <link name="rear_right_wheel_link">
     <visual><geometry><mesh filename="package://agribot_vehicle_description/generated/unity_car5/models/rear_right_wheel_visual.obj"/></geometry></visual>
-    <collision><origin rpy="1.570796326795 0 0"/><geometry><cylinder radius="0.171298325062" length="0.162000030279"/></geometry></collision>
+    <collision><origin rpy="1.570796326795 0 0"/><geometry><cylinder radius="0.429895715883" length="0.406560420044"/></geometry></collision>
   </link>
   <joint name="rear_right_wheel_joint" type="continuous">
-    <origin xyz="1.22517533896e-08 -0.202810272574 0" rpy="0 0 0"/>
+    <origin xyz="3.07473893416e-08 -0.508979099973 3.55266059304e-06" rpy="0 0 0"/>
     <parent link="base_link"/><child link="rear_right_wheel_link"/>
     <axis xyz="0 1 0"/>
