Commit message: 保存喷洒机具扩展前的多车型仿真与导航基线
保存当前六车型模型、传感器配置、规划控制适配、仿真启停和离线真机配置导出实现及开发验证记录。对应Unity配置软件提交270b192；本提交尚未添加喷洒机具。专利、软著材料与实验原始数据不纳入提交。

File: ros2_ws/src/agribot_vehicle_description/generated/ackermann_current/urdf/ackermann_current.urdf.xacro (robot description, xacro)
@@ -15,46 +15,41 @@
   </link>
   <link name="imu_link">
-    <visual><geometry><box size="0.05 0.04 0.015"/></geometry></visual>
   </link>
   <joint name="imu_mount_joint" type="fixed">
-    <origin xyz="0.14250010252 2.8882130465e-08 0.143001556396" rpy="0.00057242391631 -0.00913954898715 -2.61600803242e-06"/>
+    <origin xyz="0.142500117421 -4.16096668232e-08 0.142999082804" rpy="0.000572423858102 -0.00913954805583 -2.61646141553e-06"/>
     <parent link="base_link"/><child link="imu_link"/>
   </joint>
   <link name="lidar_link">
-    <visual><geometry><cylinder radius="0.04" length="0.08"/></geometry></visual>
   </link>
   <joint name="lidar_mount_joint" type="fixed">
-    <origin xyz="0.48000010848 1.83202484294e-08 0.233001708984" rpy="-0.00764848850667 -0.00183566112537 7.01999988451e-06"/>
+    <origin xyz="0.480000048876 -8.73142695923e-08 0.23299922049" rpy="-0.00764848897234 -0.00183566112537 7.02045099388e-06"/>
     <parent link="base_link"/><child link="lidar_link"/>
   </joint>
   <link name="right_camera_link">
-    <visual><geometry><box size="0.044 0.04 0.04"/></geometry></visual>
   </link>
   <joint name="right_camera_mount_joint" type="fixed">
-    <origin xyz="0.575500130653 -9.59825552371e-09 0.154001235962" rpy="-2.32920654986e-10 7.77125586104e-11 1.45519152284e-11"/>
+    <origin xyz="0.575500071049 -6.9207942488e-08 0.153998762369" rpy="3.98870910259e-12 3.83765547118e-10 9.01187069413e-10"/>
     <parent link="base_link"/><child link="right_camera_link"/>
   </joint>
   <link name="right_camera_optical_frame"/>
   <joint name="right_camera_measurement_joint" type="fixed">
-    <origin xyz="1.39363777407e-07 -9.59825552371e-09 1.90702087366e-06" rpy="-1.57079637051 -2.32920654986e-10 -1.57079637051"/>
+    <origin xyz="1.13671532631e-07 -6.9207942488e-08 -5.71519024106e-07" rpy="-1.57079637051 3.98870866891e-12 -1.57079637051"/>
     <parent link="right_camera_link"/><child link="right_camera_optical_frame"/>
   </joint>
   <link name="rtk_link">
-    <visual><geometry><cylinder radius="0.0225" length="0.036"/></geometry></visual>
   </link>
   <joint name="rtk_master_mount_joint" type="fixed">
-    <origin xyz="0.142500057817 0.295258492231 0.784761428833" rpy="-2.32920654986e-10 7.77125586104e-11 1.45519152284e-11"/>
+    <origin xyz="0.14250010252 0.295258432627 0.784758925438" rpy="3.98870910259e-12 3.83765547118e-10 9.01187069413e-10"/>
     <parent link="base_link"/><child link="rtk_link"/>
   </joint>
   <link name="rtk_secondary_link">
-    <visual><geometry><cylinder radius="0.0225" length="0.036"/></geometry></visual>
   </link>
   <joint name="rtk_secondary_mount_joint" type="fixed">
-    <origin xyz="0.142500087619 -0.295258432627 0.784761428833" rpy="-2.32920654986e-10 7.77125586104e-11 1.45519152284e-11"/>
+    <origin xyz="0.142500132322 -0.295258551836 0.784758925438" rpy="3.98870910259e-12 3.83765547118e-10 9.01187069413e-10"/>
     <parent link="base_link"/><child link="rtk_secondary_link"/>
   </joint>
   <link name="front_left_steering_link"/>
   <joint name="front_left_steering_joint" type="revolute">
-    <origin xyz="0.499848693609 0.294998437166 0.000669479137287" rpy="0 0 0"/>
+    <origin xyz="0.525849282742 0.294998079538 0.000502977753058" rpy="0 0 0"/>
     <parent link="base_link"/><child link="front_left_steering_link"/>
     <axis xyz="0 0 1"/>
@@ -62,5 +57,5 @@
   </joint>
   <link name="front_left_wheel_link">
-    <visual><origin rpy="1.570796326795 0 0"/><geometry><cylinder radius="0.127499997616" length="0.0814310014248"/></geometry></visual>
+    <visual><geometry><mesh filename="package://agribot_vehicle_description/generated/ackermann_current/models/front_left_wheel_visual.obj"/></geometry></visual>
     <collision><origin rpy="1.570796326795 0 0"/><geometry><cylinder radius="0.127499997616" length="0.0814310014248"/></geometry></collision>
   </link>
@@ -72,5 +67,5 @@
   <link name="front_right_steering_link"/>
   <joint name="front_right_steering_joint" type="revolute">
-    <origin xyz="0.501325964928 -0.294998288155 -0.000631332746707" rpy="0 0 0"/>
+    <origin xyz="0.527325928211 -0.294998198748 -0.000969495449681" rpy="0 0 0"/>
     <parent link="base_link"/><child link="front_right_steering_link"/>
     <axis xyz="0 0 1"/>
@@ -78,5 +73,5 @@
   </joint>
   <link name="front_right_wheel_link">
-    <visual><origin rpy="1.570796326795 0 0"/><geometry><cylinder radius="0.127499997616" length="0.0814310014248"/></geometry></visual>
+    <visual><geometry><mesh filename="package://agribot_vehicle_description/generated/ackermann_current/models/front_right_wheel_visual.obj"/></geometry></visual>
     <collision><origin rpy="1.570796326795 0 0"/><geometry><cylinder radius="0.127499997616" length="0.0814310014248"/></geometry></collision>
   </link>
@@ -87,18 +82,18 @@
   </joint>
   <link name="rear_left_wheel_link">
-    <visual><origin rpy="1.570796326795 0 0"/><geometry><cylinder radius="0.127499997616" length="0.0814310014248"/></geometry></visual>
+    <visual><geometry><mesh filename="package://agribot_vehicle_description/generated/ackermann_current/models/rear_left_wheel_visual.obj"/></geometry></visual>
     <collision><origin rpy="1.570796326795 0 0"/><geometry><cylinder radius="0.127499997616" length="0.0814310014248"/></geometry></collision>
   </link>
   <joint name="rear_left_wheel_joint" type="continuous">
-    <origin xyz="9.0567539246e-08 0.294999301434 0.000650405883789" rpy="0 0 0"/>
+    <origin xyz="4.38546038595e-07 0.29499900341 0.000733767054044" rpy="0 0 0"/>
     <parent link="base_link"/><child link="rear_left_wheel_link"/>
     <axis xyz="0 1 0"/>
   </joint>
   <link name="rear_right_wheel_link">
-    <visual><origin rpy="1.570796326795 0 0"/><geometry><cylinder radius="0.127499997616" length="0.0814310014248"/></geometry></visual>
+    <visual><geometry><mesh filename="package://agribot_vehicle_description/generated/ackermann_current/models/rear_right_wheel_visual.obj"/></geometry></visual>
     <collision><origin rpy="1.570796326795 0 0"/><geometry><cylinder radius="0.127499997616" length="0.0814310014248"/></geometry></collision>
   </link>
   <joint name="rear_right_wheel_joint" type="continuous">
-    <origin xyz="8.60191562424e-08 -0.294999241829 -0.000646591302939" rpy="0 0 0"/>
+    <origin xyz="-2.09537219575e-07 -0.294999182224 -0.000736798800062" rpy="0 0 0"/>
     <parent link="base_link"/><child link="rear_right_wheel_link"/>
     <axis xyz="0 1 0"/>
