Commit message: 保存农机资源扩展前基线：机械臂仿真、相机遮挡修复与视觉显示联动

File: ros2_ws/src/agribot_vehicle_description/generated/ackermann_current/urdf/ackermann_current.urdf.xacro (robot description, xacro)
@@ -1,101 +1,357 @@
 <?xml version="1.0"?>
-<!-- Generated by agribot_vehicle_config_tools. Do not edit by hand. -->
-<robot name="ackermann_current" xmlns:xacro="http://www.ros.org/wiki/xacro">
+<robot name="ackermann_current">
   <link name="base_link">
     <inertial>
-      <origin xyz="0.262391507626 0 0.061550501734" rpy="0 0 0"/>
-      <mass value="50"/>
-      <inertia ixx="1.91400003433" ixy="0" ixz="0" iyy="2.67199993134" iyz="0" izz="4.08400011063"/>
+      <origin xyz="0.262391507626 0 0.061550501734" rpy="0 0 0" />
+      <mass value="50" />
+      <inertia ixx="1.91400003433" ixy="0" ixz="0" iyy="2.67199993134" iyz="0" izz="4.08400011063" />
     </inertial>
-    <collision><origin xyz="0.262391507626 0 0.061550501734" rpy="0 0 0"/><geometry><box size="0.761610984802 0.631783008575 0.245800003409"/></geometry></collision>
+    <collision>
+      <origin xyz="0.262391507626 0 0.061550501734" rpy="0 0 0" />
+      <geometry>
+        <box size="0.761610984802 0.631783008575 0.245800003409" />
+      </geometry>
+    </collision>
     <visual name="vehicle_body">
-      <origin xyz="0 0 0" rpy="0 0 0"/>
-      <geometry><mesh filename="package://agribot_vehicle_description/generated/ackermann_current/models/vehicle_visual.obj" scale="1 1 1"/></geometry>
+      <origin xyz="0 0 0" rpy="0 0 0" />
+      <geometry>
+        <mesh filename="package://agribot_vehicle_description/generated/ackermann_current/models/vehicle_visual.obj" scale="1 1 1" />
+      </geometry>
     </visual>
   </link>
   <link name="imu_link">
+    <visual>
+      <geometry>
+        <mesh filename="package://agribot_vehicle_description/generated/ackermann_current/models/sensor_imu_visual.obj" />
+      </geometry>
+    </visual>
   </link>
   <joint name="imu_mount_joint" type="fixed">
-    <origin xyz="0.142500117421 -4.16096668232e-08 0.142999082804" rpy="0.000572423858102 -0.00913954805583 -2.61646141553e-06"/>
-    <parent link="base_link"/><child link="imu_link"/>
+    <origin xyz="0.142499953508 1.09291818262e-07 0.142997741699" rpy="0.000572424090933 -0.00913954898715 -2.61600916929e-06" />
+    <parent link="base_link" />
+    <child link="imu_link" />
   </joint>
   <link name="lidar_link">
+    <visual>
+      <geometry>
+        <mesh filename="package://agribot_vehicle_description/generated/ackermann_current/models/sensor_lidar_visual.obj" />
+      </geometry>
+    </visual>
   </link>
   <joint name="lidar_mount_joint" type="fixed">
-    <origin xyz="0.480000048876 -8.73142695923e-08 0.23299922049" rpy="-0.00764848897234 -0.00183566112537 7.02045099388e-06"/>
-    <parent link="base_link"/><child link="lidar_link"/>
+    <origin xyz="0.479999929667 7.1564620896e-08 0.232997894287" rpy="-0.00764848804101 -0.00183566054329 7.01999897501e-06" />
+    <parent link="base_link" />
+    <child link="lidar_link" />
   </joint>
   <link name="right_camera_link">
+    <visual>
+      <geometry>
+        <mesh filename="package://agribot_vehicle_description/generated/ackermann_current/models/sensor_right_camera_visual.obj" />
+      </geometry>
+    </visual>
   </link>
   <joint name="right_camera_mount_joint" type="fixed">
-    <origin xyz="0.575500071049 -6.9207942488e-08 0.153998762369" rpy="3.98870910259e-12 3.83765547118e-10 9.01187069413e-10"/>
-    <parent link="base_link"/><child link="right_camera_link"/>
-  </joint>
-  <link name="right_camera_optical_frame"/>
+    <origin xyz="0.575500011444 9.52900123252e-08 0.153997421265" rpy="0 3.54046791884e-10 0" />
+    <parent link="base_link" />
+    <child link="right_camera_link" />
+  </joint>
+  <link name="right_camera_optical_frame" />
   <joint name="right_camera_measurement_joint" type="fixed">
-    <origin xyz="1.13671532631e-07 -6.9207942488e-08 -5.71519024106e-07" rpy="-1.57079637051 3.98870866891e-12 -1.57079637051"/>
-    <parent link="right_camera_link"/><child link="right_camera_optical_frame"/>
+    <origin xyz="8.74736727496e-09 9.52900123252e-08 -1.90754212781e-06" rpy="-1.57079637051 0 -1.57079637051" />
+    <parent link="right_camera_link" />
+    <child link="right_camera_optical_frame" />
   </joint>
   <link name="rtk_link">
+    <visual>
+      <geometry>
+        <mesh filename="package://agribot_vehicle_description/generated/ackermann_current/models/sensor_rtk_master_visual.obj" />
+      </geometry>
+    </visual>
   </link>
   <joint name="rtk_master_mount_joint" type="fixed">
-    <origin xyz="0.14250010252 0.295258432627 0.784758925438" rpy="3.98870910259e-12 3.83765547118e-10 9.01187069413e-10"/>
-    <parent link="base_link"/><child link="rtk_link"/>
+    <origin xyz="0.142499923706 0.295258581638 0.784757614136" rpy="0 3.54046791884e-10 0" />
+    <parent link="base_link" />
+    <child link="rtk_link" />
   </joint>
   <link name="rtk_secondary_link">
   </link>
   <joint name="rtk_secondary_mount_joint" type="fixed">
-    <origin xyz="0.142500132322 -0.295258551836 0.784758925438" rpy="3.98870910259e-12 3.83765547118e-10 9.01187069413e-10"/>
-    <parent link="base_link"/><child link="rtk_secondary_link"/>
-  </joint>
-  <link name="front_left_steering_link"/>
+    <origin xyz="0.142499923706 -0.295258373022 0.784757614136" rpy="0 3.54046791884e-10 0" />
+    <parent link="base_link" />
+    <child link="rtk_secondary_link" />
+  </joint>
+  <link name="front_left_steering_link" />
   <joint name="front_left_steering_joint" type="revolute">
-    <origin xyz="0.525849282742 0.294998079538 0.000502977753058" rpy="0 0 0"/>
-    <parent link="base_link"/><child link="front_left_steering_link"/>
-    <axis xyz="0 0 1"/>
-    <limit lower="-0.384000003338" upper="0.384000003338" effort="200" velocity="1.5"/>
+    <origin xyz="0.525849163532 0.294998288155 0.000398635689635" rpy="0 0 0" />
+    <parent link="base_link" />
+    <child link="front_left_steering_link" />
+    <axis xyz="0 0 1" />
+    <limit lower="-0.384000003338" upper="0.384000003338" effort="200" velocity="1.5" />
   </joint>
   <link name="front_left_wheel_link">
-    <visual><geometry><mesh filename="package://agribot_vehicle_description/generated/ackermann_current/models/front_left_wheel_visual.obj"/></geometry></visual>
-    <collision><origin rpy="1.570796326795 0 0"/><geometry><cylinder radius="0.127499997616" length="0.0814310014248"/></geometry></collision>
+    <visual>
+      <geometry>
+        <mesh filename="package://agribot_vehicle_description/generated/ackermann_current/models/front_left_wheel_visual.obj" />
+      </geometry>
+    </visual>
+    <collision>
+      <origin rpy="1.570796326795 0 0" />
+      <geometry>
+        <cylinder radius="0.127499997616" length="0.0814310014248" />
+      </geometry>
+    </collision>
   </link>
   <joint name="front_left_wheel_joint" type="continuous">
-    <origin xyz="0 0 0" rpy="0 0 0"/>
-    <parent link="front_left_steering_link"/><child link="front_left_wheel_link"/>
-    <axis xyz="0 1 0"/>
-  </joint>
-  <link name="front_right_steering_link"/>
+    <origin xyz="0 0 0" rpy="0 0 0" />
+    <parent link="front_left_steering_link" />
+    <child link="front_left_wheel_link" />
+    <axis xyz="0 1 0" />
+  </joint>
+  <link name="front_right_steering_link" />
   <joint name="front_right_steering_joint" type="revolute">
-    <origin xyz="0.527325928211 -0.294998198748 -0.000969495449681" rpy="0 0 0"/>
-    <parent link="base_link"/><child link="front_right_steering_link"/>
-    <axis xyz="0 0 1"/>
-    <limit lower="-0.384000003338" upper="0.384000003338" effort="200" velocity="1.5"/>
+    <origin xyz="0.527325689793 -0.294998109341 -0.000999450916424" rpy="0 0 0" />
+    <parent link="base_link" />
+    <child link="front_right_steering_link" />
+    <axis xyz="0 0 1" />
+    <limit lower="-0.384000003338" upper="0.384000003338" effort="200" velocity="1.5" />
   </joint>
   <link name="front_right_wheel_link">
-    <visual><geometry><mesh filename="package://agribot_vehicle_description/generated/ackermann_current/models/front_right_wheel_visual.obj"/></geometry></visual>
-    <collision><origin rpy="1.570796326795 0 0"/><geometry><cylinder radius="0.127499997616" length="0.0814310014248"/></geometry></collision>
+    <visual>
+      <geometry>
+        <mesh filename="package://agribot_vehicle_description/generated/ackermann_current/models/front_right_wheel_visual.obj" />
+      </geometry>
+    </visual>
+    <collision>
+      <origin rpy="1.570796326795 0 0" />
+      <geometry>
+        <cylinder radius="0.127499997616" length="0.0814310014248" />
+      </geometry>
+    </collision>
   </link>
   <joint name="front_right_wheel_joint" type="continuous">
-    <origin xyz="0 0 0" rpy="0 0 0"/>
-    <parent link="front_right_steering_link"/><child link="front_right_wheel_link"/>
-    <axis xyz="0 1 0"/>
+    <origin xyz="0 0 0" rpy="0 0 0" />
+    <parent link="front_right_steering_link" />
+    <child link="front_right_wheel_link" />
+    <axis xyz="0 1 0" />
   </joint>
   <link name="rear_left_wheel_link">
-    <visual><geometry><mesh filename="package://agribot_vehicle_description/generated/ackermann_current/models/rear_left_wheel_visual.obj"/></geometry></visual>
-    <collision><origin rpy="1.570796326795 0 0"/><geometry><cylinder radius="0.127499997616" length="0.0814310014248"/></geometry></collision>
+    <visual>
+      <geometry>
+        <mesh filename="package://agribot_vehicle_description/generated/ackermann_current/models/rear_left_wheel_visual.obj" />
+      </geometry>
+    </visual>
+    <collision>
+      <origin rpy="1.570796326795 0 0" />
+      <geometry>
+        <cylinder radius="0.127499997616" length="0.0814310014248" />
+      </geometry>
+    </collision>
   </link>
   <joint name="rear_left_wheel_joint" type="continuous">
-    <origin xyz="4.38546038595e-07 0.29499900341 0.000733767054044" rpy="0 0 0"/>
-    <parent link="base_link"/><child link="rear_left_wheel_link"/>
-    <axis xyz="0 1 0"/>
+    <origin xyz="3.90425213936e-07 0.294999241829 0.000696182192769" rpy="0 0 0" />
+    <parent link="base_link" />
+    <child link="rear_left_wheel_link" />
+    <axis xyz="0 1 0" />
   </joint>
   <link name="rear_right_wheel_link">
-    <visual><geometry><mesh filename="package://agribot_vehicle_description/generated/ackermann_current/models/rear_right_wheel_visual.obj"/></geometry></visual>
-    <collision><origin rpy="1.570796326795 0 0"/><geometry><cylinder radius="0.127499997616" length="0.0814310014248"/></geometry></collision>
+    <visual>
+      <geometry>
+        <mesh filename="package://agribot_vehicle_description/generated/ackermann_current/models/rear_right_wheel_visual.obj" />
+      </geometry>
+    </visual>
+    <collision>
+      <origin rpy="1.570796326795 0 0" />
+      <geometry>
+        <cylinder radius="0.127499997616" length="0.0814310014248" />
+      </geometry>
+    </collision>
   </link>
   <joint name="rear_right_wheel_joint" type="continuous">
-    <origin xyz="-2.09537219575e-07 -0.294999182224 -0.000736798800062" rpy="0 0 0"/>
-    <parent link="base_link"/><child link="rear_right_wheel_link"/>
-    <axis xyz="0 1 0"/>
+    <origin xyz="-4.17683509113e-07 -0.294999063015 -0.00069999700645" rpy="0 0 0" />
+    <parent link="base_link" />
+    <child link="rear_right_wheel_link" />
+    <axis xyz="0 1 0" />
+  </joint>
+  <link name="manipulator_link_base">
+    <visual>
+      <origin xyz="0 0 0" rpy="0 0 0" />
+      <geometry>
+        <mesh filename="package://agribot_manipulator_sim/models/lite6/meshes/link_base.stl" />
+      </geometry>
+      <material name="manipulator_link_base_material">
+        <color rgba="0.85 0.88 0.90 1" />
+      </material>
+    </visual>
+  </link>
+  <link name="manipulator_link1">
+    <visual>
+      <origin xyz="0 0 0" rpy="0 0 0" />
+      <geometry>
+        <mesh filename="package://agribot_manipulator_sim/models/lite6/meshes/link1.stl" />
+      </geometry>
+      <material name="manipulator_link1_material">
+        <color rgba="0.85 0.88 0.90 1" />
+      </material>
+    </visual>
+  </link>
+  <link name="manipulator_link2">
+    <visual>
+      <origin xyz="0 0 0" rpy="0 0 0" />
+      <geometry>
+        <mesh filename="package://agribot_manipulator_sim/models/lite6/meshes/link2.stl" />
+      </geometry>
+      <material name="manipulator_link2_material">
+        <color rgba="0.85 0.88 0.90 1" />
+      </material>
+    </visual>
+  </link>
+  <link name="manipulator_link3">
+    <visual>
+      <origin xyz="0 0 0" rpy="0 0 0" />
+      <geometry>
+        <mesh filename="package://agribot_manipulator_sim/models/lite6/meshes/link3.stl" />
+      </geometry>
+      <material name="manipulator_link3_material">
+        <color rgba="0.85 0.88 0.90 1" />
+      </material>
+    </visual>
+  </link>
+  <link name="manipulator_link4">
+    <visual>
+      <origin xyz="0 0 0" rpy="0 0 0" />
+      <geometry>
+        <mesh filename="package://agribot_manipulator_sim/models/lite6/meshes/link4.stl" />
+      </geometry>
+      <material name="manipulator_link4_material">
+        <color rgba="0.85 0.88 0.90 1" />
+      </material>
+    </visual>
+  </link>
+  <link name="manipulator_link5">
+    <visual>
+      <origin xyz="0 0 0" rpy="0 0 0" />
+      <geometry>
+        <mesh filename="package://agribot_manipulator_sim/models/lite6/meshes/link5.stl" />
+      </geometry>
+      <material name="manipulator_link5_material">
+        <color rgba="0.85 0.88 0.90 1" />
+      </material>
+    </visual>
+  </link>
+  <link name="manipulator_link6">
+    <visual>
+      <origin xyz="0 0 0" rpy="0 0 0" />
+      <geometry>
+        <mesh filename="package://agribot_manipulator_sim/models/lite6/meshes/link6.stl" />
+      </geometry>
+      <material name="manipulator_link6_material">
+        <color rgba="0.60 0.64 0.68 1" />
+      </material>
+    </visual>
+  </link>
+  <link name="manipulator_gripper_shell">
+    <visual>
+      <origin xyz="0 0 0" rpy="0 0 0" />
+      <geometry>
+        <mesh filename="package://agribot_manipulator_sim/models/lite6/meshes/gripper_shell.stl" />
+      </geometry>
+      <material name="manipulator_gripper_shell_material">
+        <color rgba="0.85 0.88 0.90 1" />
+      </material>
+    </visual>
+  </link>
+  <link name="manipulator_finger1">
+    <visual>
+      <origin xyz="0 0 0" rpy="0 0 0" />
+      <geometry>
+        <mesh filename="package://agribot_manipulator_sim/models/lite6/meshes/finger1.stl" />
+      </geometry>
+      <material name="manipulator_finger1_material">
+        <color rgba="0.20 0.22 0.24 1" />
+      </material>
+    </visual>
+  </link>
+  <link name="manipulator_finger2">
+    <visual>
+      <origin xyz="0 0 0" rpy="0 0 0" />
+      <geometry>
+        <mesh filename="package://agribot_manipulator_sim/models/lite6/meshes/finger2.stl" />
+      </geometry>
+      <material name="manipulator_finger2_material">
+        <color rgba="0.20 0.22 0.24 1" />
+      </material>
+    </visual>
+  </link>
+  <joint name="manipulator_mount_joint" type="fixed">
+    <parent link="base_link" />
+    <child link="manipulator_link_base" />
+    <origin xyz="0.2527782023 0.0006425103056 0.1394004822" rpy="0.002361407736 0.003225819673 6.398016922e-06" />
+  </joint>
+  <joint name="manipulator_joint1" type="revolute">
+    <parent link="manipulator_link_base" />
+    <child link="manipulator_link1" />
+    <origin xyz="0 0 0.2435" rpy="0 0 0" />
+    <axis xyz="0 0 1" />
+    <limit lower="-6.283185307179586" upper="6.283185307179586" effort="50" velocity="3.14" />
+    <dynamics damping="1.0" friction="1.0" />
+  </joint>
+  <joint name="manipulator_joint2" type="revolute">
+    <parent link="manipulator_link1" />
+    <child link="manipulator_link2" />
+    <origin xyz="0 0 0" rpy="1.5708 -1.5708 3.1416" />
+    <axis xyz="0 0 1" />
+    <limit lower="-2.61799" upper="2.61799" effort="50" velocity="3.14" />
+    <dynamics damping="1.0" friction="1.0" />
+  </joint>
+  <joint name="manipulator_joint3" type="revolute">
+    <parent link="manipulator_link2" />
+    <child link="manipulator_link3" />
+    <origin xyz="0.2002 0 0" rpy="-3.1416 0 1.5708" />
+    <axis xyz="0 0 1" />
+    <limit lower="-0.061087" upper="5.235988" effort="50" velocity="3.14" />
+    <dynamics damping="1.0" friction="1.0" />
+  </joint>
+  <joint name="manipulator_joint4" type="revolute">
+    <parent link="manipulator_link3" />
+    <child link="manipulator_link4" />
+    <origin xyz="0.087 -0.22761 0" rpy="1.5708 0 0" />
+    <axis xyz="0 0 1" />
+    <limit lower="-6.283185307179586" upper="6.283185307179586" effort="50" velocity="3.14" />
+    <dynamics damping="1.0" friction="1.0" />
+  </joint>
+  <joint name="manipulator_joint5" type="revolute">
+    <parent link="manipulator_link4" />
+    <child link="manipulator_link5" />
+    <origin xyz="0 0 0" rpy="1.5708 0 0" />
+    <axis xyz="0 0 1" />
+    <limit lower="-2.1642" upper="2.1642" effort="50" velocity="3.14" />
+    <dynamics damping="1.0" friction="1.0" />
+  </joint>
+  <joint name="manipulator_joint6" type="revolute">
+    <parent link="manipulator_link5" />
+    <child link="manipulator_link6" />
+    <origin xyz="0 0.0625 0" rpy="-1.5708 0 0" />
+    <axis xyz="0 0 1" />
+    <limit lower="-6.283185307179586" upper="6.283185307179586" effort="50" velocity="3.14" />
+    <dynamics damping="1.0" friction="1.0" />
+  </joint>
+  <joint name="manipulator_gripper_mount" type="fixed">
+    <parent link="manipulator_link6" />
+    <child link="manipulator_gripper_shell" />
+    <origin xyz="0 0 0" rpy="0 0 0" />
+  </joint>
+  <joint name="manipulator_finger_joint1" type="prismatic">
+    <parent link="manipulator_gripper_shell" />
+    <child link="manipulator_finger1" />
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
File: ros2_ws/src/agribot_vehicle_description/generated/unity_car1/urdf/unity_car1.urdf.xacro (robot description, xacro)
@@ -4,9 +4,9 @@
   <link name="base_link">
     <inertial>
-      <origin xyz="0.312528043985 5.96046447754e-08 0.230181902647" rpy="0 0 0"/>
+      <origin xyz="0.312528043985 5.96046447754e-08 0.230182856321" rpy="0 0 0"/>
       <mass value="50"/>
-      <inertia ixx="3.90098214149" ixy="0" ixz="0" iyy="8.18287086487" iyz="0" izz="7.67456102371"/>
+      <inertia ixx="3.90099358559" ixy="0" ixz="0" iyy="8.18288230896" iyz="0" izz="7.67456102371"/>
     </inertial>
-    <collision><origin xyz="0.312528043985 5.96046447754e-08 0.230181902647" rpy="0 0 0"/><geometry><box size="1.19782054424 0.638060092926 0.727402925491"/></geometry></collision>
+    <collision><origin xyz="0.312528043985 5.96046447754e-08 0.230182856321" rpy="0 0 0"/><geometry><box size="1.19782054424 0.638060092926 0.72740483284"/></geometry></collision>
     <visual name="vehicle_body">
       <origin xyz="0 0 0" rpy="0 0 0"/>
@@ -25,5 +25,5 @@
   </link>
   <joint name="lidar_mount_joint" type="fixed">
-    <origin xyz="0.243228211999 0.00300005986355 0.573192596436" rpy="0 0 0"/>
+    <origin xyz="0.285124033689 0.00303386058658 0.572944641113" rpy="0 0 0"/>
     <parent link="base_link"/><child link="lidar_link"/>
   </joint>
@@ -44,5 +44,5 @@
   </link>
   <joint name="rtk_master_mount_joint" type="fixed">
-    <origin xyz="0.105528108776 0.334000945091 1.05739212036" rpy="0 0 0"/>
+    <origin xyz="0.180623948574 0.334000825882 1.05604362488" rpy="0 0 0"/>
     <parent link="base_link"/><child link="rtk_link"/>
   </joint>
@@ -50,5 +50,5 @@
   </link>
   <joint name="rtk_secondary_mount_joint" type="fixed">
-    <origin xyz="0.105528242886 -0.316000789404 1.05739212036" rpy="0 0 0"/>
+    <origin xyz="0.18062402308 -0.316000819206 1.05604362488" rpy="0 0 0"/>
     <parent link="base_link"/><child link="rtk_secondary_link"/>
   </joint>
