Commit message: 保存农机资源扩展前基线：机械臂仿真、相机遮挡修复与视觉显示联动

File: ros2_ws/src/agribot_vehicle_description/generated/unity_car3/urdf/unity_car3.urdf.xacro (robot description, xacro)
@@ -1,87 +1,321 @@
 <?xml version="1.0"?>
-<!-- Generated by agribot_vehicle_config_tools. Do not edit by hand. -->
-<robot name="unity_car3" xmlns:xacro="http://www.ros.org/wiki/xacro">
+<robot name="unity_car3">
   <link name="base_link">
     <inertial>
-      <origin xyz="0.0630367994308 0.00308442115784 0.256492316723" rpy="0 0 0"/>
-      <mass value="50"/>
-      <inertia ixx="5.03856372833" ixy="0" ixz="0" iyy="8.07163715363" iyz="0" izz="7.73918104172"/>
+      <origin xyz="0.0630367994308 0.00308442115784 0.256492316723" rpy="0 0 0" />
+      <mass value="50" />
+      <inertia ixx="5.03856372833" ixy="0" ixz="0" iyy="8.07163715363" iyz="0" izz="7.73918104172" />
     </inertial>
-    <collision><origin xyz="0.0630367994308 0.00308442115784 0.256492316723" rpy="0 0 0"/><geometry><box size="1.13695669174 0.751487195492 0.802821516991"/></geometry></collision>
+    <collision>
+      <origin xyz="0.0630367994308 0.00308442115784 0.256492316723" rpy="0 0 0" />
+      <geometry>
+        <box size="1.13695669174 0.751487195492 0.802821516991" />
+      </geometry>
+    </collision>
     <visual name="vehicle_body">
-      <origin xyz="0 0 0" rpy="0 0 0"/>
-      <geometry><mesh filename="package://agribot_vehicle_description/generated/unity_car3/models/vehicle_visual.obj" scale="1 1 1"/></geometry>
+      <origin xyz="0 0 0" rpy="0 0 0" />
+      <geometry>
+        <mesh filename="package://agribot_vehicle_description/generated/unity_car3/models/vehicle_visual.obj" scale="1 1 1" />
+      </geometry>
     </visual>
   </link>
   <link name="imu_link">
-    <visual><geometry><mesh filename="package://agribot_vehicle_description/generated/unity_car3/models/sensor_imu_visual.obj"/></geometry></visual>
+    <visual>
+      <geometry>
+        <mesh filename="package://agribot_vehicle_description/generated/unity_car3/models/sensor_imu_visual.obj" />
+      </geometry>
+    </visual>
   </link>
   <joint name="imu_mount_joint" type="fixed">
-    <origin xyz="0.422795921564 0.113218359649 0.668453216553" rpy="0 0 0"/>
-    <parent link="base_link"/><child link="imu_link"/>
+    <origin xyz="0.422795921564 0.113218359649 0.668453216553" rpy="0 0 0" />
+    <parent link="base_link" />
+    <child link="imu_link" />
   </joint>
   <link name="lidar_link">
-    <visual><geometry><mesh filename="package://agribot_vehicle_description/generated/unity_car3/models/sensor_lidar_visual.obj"/></geometry></visual>
+    <visual>
+      <geometry>
+        <mesh filename="package://agribot_vehicle_description/generated/unity_car3/models/sensor_lidar_visual.obj" />
+      </geometry>
+    </visual>
   </link>
   <joint name="lidar_mount_joint" type="fixed">
-    <origin xyz="0.480195939541 -0.00778169976547 0.697454452515" rpy="0 0 0"/>
-    <parent link="base_link"/><child link="lidar_link"/>
+    <origin xyz="0.480195939541 -0.00778169976547 0.697454452515" rpy="0 0 0" />
+    <parent link="base_link" />
+    <child link="lidar_link" />
   </joint>
   <link name="right_camera_link">
-    <visual><geometry><mesh filename="package://agribot_vehicle_description/generated/unity_car3/models/sensor_right_camera_visual.obj"/></geometry></visual>
+    <visual>
+      <geometry>
+        <mesh filename="package://agribot_vehicle_description/generated/unity_car3/models/sensor_right_camera_visual.obj" />
+      </geometry>
+    </visual>
   </link>
   <joint name="right_camera_mount_joint" type="fixed">
-    <origin xyz="0.495695948601 -0.00708170095459 0.799753189087" rpy="0 0 0"/>
-    <parent link="base_link"/><child link="right_camera_link"/>
-  </joint>
-  <link name="right_camera_optical_frame"/>
+    <origin xyz="0.495695948601 -0.00708170095459 0.799753189087" rpy="0 0 0" />
+    <parent link="base_link" />
+    <child link="right_camera_link" />
+  </joint>
+  <link name="right_camera_optical_frame" />
   <joint name="right_camera_measurement_joint" type="fixed">
-    <origin xyz="1.08225592044e-07 4.61971438881e-08 0" rpy="-1.57079637051 0 -1.57079637051"/>
-    <parent link="right_camera_link"/><child link="right_camera_optical_frame"/>
+    <origin xyz="1.08225592044e-07 4.61971438881e-08 0" rpy="-1.57079637051 0 -1.57079637051" />
+    <parent link="right_camera_link" />
+    <child link="right_camera_optical_frame" />
   </joint>
   <link name="rtk_link">
-    <visual><geometry><mesh filename="package://agribot_vehicle_description/generated/unity_car3/models/sensor_rtk_master_visual.obj"/></geometry></visual>
+    <visual>
+      <geometry>
+        <mesh filename="package://agribot_vehicle_description/generated/unity_car3/models/sensor_rtk_master_visual.obj" />
+      </geometry>
+    </visual>
   </link>
   <joint name="rtk_master_mount_joint" type="fixed">
-    <origin xyz="-0.103804320097 0.326218962669 0.946853637695" rpy="0 0 0"/>
-    <parent link="base_link"/><child link="rtk_link"/>
+    <origin xyz="0.0481957346201 0.326219111681 0.946853637695" rpy="0 0 0" />
+    <parent link="base_link" />
+    <child link="rtk_link" />
   </joint>
   <link name="rtk_secondary_link">
   </link>
   <joint name="rtk_secondary_mount_joint" type="fixed">
-    <origin xyz="-0.103804215789 -0.323782622814 0.946853637695" rpy="0 0 0"/>
-    <parent link="base_link"/><child link="rtk_secondary_link"/>
+    <origin xyz="0.0481958426535 -0.32378256321 0.946853637695" rpy="0 0 0" />
+    <parent link="base_link" />
+    <child link="rtk_secondary_link" />
   </joint>
   <link name="front_left_wheel_link">
-    <collision><origin rpy="1.570796326795 0 0"/><geometry><cylinder radius="0.224918439984" length="0.154119610786"/></geometry></collision>
+    <collision>
+      <origin rpy="1.570796326795 0 0" />
+      <geometry>
+        <cylinder radius="0.224918439984" length="0.154119610786" />
+      </geometry>
+    </collision>
   </link>
   <joint name="front_left_wheel_joint" type="continuous">
-    <origin xyz="0.200999945402 0.294500052929 0" rpy="0 0 0"/>
-    <parent link="base_link"/><child link="front_left_wheel_link"/>
-    <axis xyz="0 1 0"/>
+    <origin xyz="0.200999945402 0.294500052929 0" rpy="0 0 0" />
+    <parent link="base_link" />
+    <child link="front_left_wheel_link" />
+    <axis xyz="0 1 0" />
   </joint>
   <link name="front_right_wheel_link">
-    <collision><origin rpy="1.570796326795 0 0"/><geometry><cylinder radius="0.224918439984" length="0.154119729996"/></geometry></collision>
+    <collision>
+      <origin rpy="1.570796326795 0 0" />
+      <geometry>
+        <cylinder radius="0.224918439984" length="0.154119729996" />
+      </geometry>
+    </collision>
   </link>
   <joint name="front_right_wheel_joint" type="continuous">
-    <origin xyz="0.201000019908 -0.294500023127 0" rpy="0 0 0"/>
-    <parent link="base_link"/><child link="front_right_wheel_link"/>
-    <axis xyz="0 1 0"/>
+    <origin xyz="0.201000019908 -0.294500023127 0" rpy="0 0 0" />
+    <parent link="base_link" />
+    <child link="front_right_wheel_link" />
+    <axis xyz="0 1 0" />
   </joint>
   <link name="rear_left_wheel_link">
-    <collision><origin rpy="1.570796326795 0 0"/><geometry><cylinder radius="0.224918439984" length="0.154119610786"/></geometry></collision>
+    <collision>
+      <origin rpy="1.570796326795 0 0" />
+      <geometry>
+        <cylinder radius="0.224918439984" length="0.154119610786" />
+      </geometry>
+    </collision>
   </link>
   <joint name="rear_left_wheel_joint" type="continuous">
-    <origin xyz="-0.201000079513 0.294499993324 0" rpy="0 0 0"/>
-    <parent link="base_link"/><child link="rear_left_wheel_link"/>
-    <axis xyz="0 1 0"/>
+    <origin xyz="-0.201000079513 0.294499993324 0" rpy="0 0 0" />
+    <parent link="base_link" />
+    <child link="rear_left_wheel_link" />
+    <axis xyz="0 1 0" />
   </joint>
   <link name="rear_right_wheel_link">
-    <collision><origin rpy="1.570796326795 0 0"/><geometry><cylinder radius="0.224918439984" length="0.154119610786"/></geometry></collision>
+    <collision>
+      <origin rpy="1.570796326795 0 0" />
+      <geometry>
+        <cylinder radius="0.224918439984" length="0.154119610786" />
+      </geometry>
+    </collision>
   </link>
   <joint name="rear_right_wheel_joint" type="continuous">
-    <origin xyz="-0.201000005007 -0.294500052929 0" rpy="0 0 0"/>
-    <parent link="base_link"/><child link="rear_right_wheel_link"/>
-    <axis xyz="0 1 0"/>
+    <origin xyz="-0.201000005007 -0.294500052929 0" rpy="0 0 0" />
+    <parent link="base_link" />
+    <child link="rear_right_wheel_link" />
+    <axis xyz="0 1 0" />
+  </joint>
+  <link name="manipulator_link_base">
+    <visual>
+      <origin xyz="0 0 0" rpy="0 0 0" />
+      <geometry>
+        <mesh filename="package://agribot_manipulator_sim/models/lite6/meshes/link_base.stl" />
+      </geometry>
+      <material name="manipulator_link_base_material">
+        <color rgba="0.85 0.88 0.90 1" />
+      </material>
+    </visual>
+  </link>
+  <link name="manipulator_link1">
+    <visual>
+      <origin xyz="0 0 0" rpy="0 0 0" />
+      <geometry>
+        <mesh filename="package://agribot_manipulator_sim/models/lite6/meshes/link1.stl" />
+      </geometry>
+      <material name="manipulator_link1_material">
+        <color rgba="0.85 0.88 0.90 1" />
+      </material>
+    </visual>
+  </link>
+  <link name="manipulator_link2">
+    <visual>
+      <origin xyz="0 0 0" rpy="0 0 0" />
+      <geometry>
+        <mesh filename="package://agribot_manipulator_sim/models/lite6/meshes/link2.stl" />
+      </geometry>
+      <material name="manipulator_link2_material">
+        <color rgba="0.85 0.88 0.90 1" />
+      </material>
+    </visual>
+  </link>
+  <link name="manipulator_link3">
+    <visual>
+      <origin xyz="0 0 0" rpy="0 0 0" />
+      <geometry>
+        <mesh filename="package://agribot_manipulator_sim/models/lite6/meshes/link3.stl" />
+      </geometry>
+      <material name="manipulator_link3_material">
+        <color rgba="0.85 0.88 0.90 1" />
+      </material>
+    </visual>
+  </link>
+  <link name="manipulator_link4">
+    <visual>
+      <origin xyz="0 0 0" rpy="0 0 0" />
+      <geometry>
+        <mesh filename="package://agribot_manipulator_sim/models/lite6/meshes/link4.stl" />
+      </geometry>
+      <material name="manipulator_link4_material">
+        <color rgba="0.85 0.88 0.90 1" />
+      </material>
+    </visual>
+  </link>
+  <link name="manipulator_link5">
+    <visual>
+      <origin xyz="0 0 0" rpy="0 0 0" />
+      <geometry>
+        <mesh filename="package://agribot_manipulator_sim/models/lite6/meshes/link5.stl" />
+      </geometry>
+      <material name="manipulator_link5_material">
+        <color rgba="0.85 0.88 0.90 1" />
+      </material>
+    </visual>
+  </link>
+  <link name="manipulator_link6">
+    <visual>
+      <origin xyz="0 0 0" rpy="0 0 0" />
+      <geometry>
+        <mesh filename="package://agribot_manipulator_sim/models/lite6/meshes/link6.stl" />
+      </geometry>
+      <material name="manipulator_link6_material">
+        <color rgba="0.60 0.64 0.68 1" />
+      </material>
+    </visual>
+  </link>
+  <link name="manipulator_gripper_shell">
+    <visual>
+      <origin xyz="0 0 0" rpy="0 0 0" />
+      <geometry>
+        <mesh filename="package://agribot_manipulator_sim/models/lite6/meshes/gripper_shell.stl" />
+      </geometry>
+      <material name="manipulator_gripper_shell_material">
+        <color rgba="0.85 0.88 0.90 1" />
+      </material>
+    </visual>
+  </link>
+  <link name="manipulator_finger1">
+    <visual>
+      <origin xyz="0 0 0" rpy="0 0 0" />
+      <geometry>
+        <mesh filename="package://agribot_manipulator_sim/models/lite6/meshes/finger1.stl" />
+      </geometry>
+      <material name="manipulator_finger1_material">
+        <color rgba="0.20 0.22 0.24 1" />
+      </material>
+    </visual>
+  </link>
+  <link name="manipulator_finger2">
+    <visual>
+      <origin xyz="0 0 0" rpy="0 0 0" />
+      <geometry>
+        <mesh filename="package://agribot_manipulator_sim/models/lite6/meshes/finger2.stl" />
+      </geometry>
+      <material name="manipulator_finger2_material">
+        <color rgba="0.20 0.22 0.24 1" />
+      </material>
+    </visual>
+  </link>
+  <joint name="manipulator_mount_joint" type="fixed">
+    <parent link="base_link" />
+    <child link="manipulator_link_base" />
+    <origin xyz="-0.2136621326 0.03248455748 0.4266700745" rpy="0 1.192092896e-07 1.192092753e-07" />
+  </joint>
+  <joint name="manipulator_joint1" type="revolute">
+    <parent link="manipulator_link_base" />
+    <child link="manipulator_link1" />
+    <origin xyz="0 0 0.2435" rpy="0 0 0" />
+    <axis xyz="0 0 1" />
+    <limit lower="-6.283185307179586" upper="6.283185307179586" effort="50" velocity="3.14" />
+    <dynamics damping="1.0" friction="1.0" />
+  </joint>
+  <joint name="manipulator_joint2" type="revolute">
+    <parent link="manipulator_link1" />
+    <child link="manipulator_link2" />
+    <origin xyz="0 0 0" rpy="1.5708 -1.5708 3.1416" />
+    <axis xyz="0 0 1" />
+    <limit lower="-2.61799" upper="2.61799" effort="50" velocity="3.14" />
+    <dynamics damping="1.0" friction="1.0" />
+  </joint>
+  <joint name="manipulator_joint3" type="revolute">
+    <parent link="manipulator_link2" />
+    <child link="manipulator_link3" />
+    <origin xyz="0.2002 0 0" rpy="-3.1416 0 1.5708" />
+    <axis xyz="0 0 1" />
+    <limit lower="-0.061087" upper="5.235988" effort="50" velocity="3.14" />
+    <dynamics damping="1.0" friction="1.0" />
+  </joint>
+  <joint name="manipulator_joint4" type="revolute">
+    <parent link="manipulator_link3" />
+    <child link="manipulator_link4" />
+    <origin xyz="0.087 -0.22761 0" rpy="1.5708 0 0" />
+    <axis xyz="0 0 1" />
+    <limit lower="-6.283185307179586" upper="6.283185307179586" effort="50" velocity="3.14" />
+    <dynamics damping="1.0" friction="1.0" />
+  </joint>
+  <joint name="manipulator_joint5" type="revolute">
+    <parent link="manipulator_link4" />
+    <child link="manipulator_link5" />
+    <origin xyz="0 0 0" rpy="1.5708 0 0" />
+    <axis xyz="0 0 1" />
+    <limit lower="-2.1642" upper="2.1642" effort="50" velocity="3.14" />
+    <dynamics damping="1.0" friction="1.0" />
+  </joint>
+  <joint name="manipulator_joint6" type="revolute">
+    <parent link="manipulator_link5" />
+    <child link="manipulator_link6" />
+    <origin xyz="0 0.0625 0" rpy="-1.5708 0 0" />
+    <axis xyz="0 0 1" />
+    <limit lower="-6.283185307179586" upper="6.283185307179586" effort="50" velocity="3.14" />
+    <dynamics damping="1.0" friction="1.0" />
+  </joint>
+  <joint name="manipulator_gripper_mount" type="fixed">
+    <parent link="manipulator_link6" />
+    <child link="manipulator_gripper_shell" />
+    <origin xyz="0 0 0" rpy="0 0 0" />
+  </joint>
+  <joint name="manipulator_finger_joint1" type="prismatic">
+    <parent link="manipulator_gripper_shell" />
+    <child link="manipulator_finger1" />
+    <origin xyz="0 0 0.0543" rpy="0 0 0" />
+    <axis xyz="0 1 0" />
+    <limit lower="0" upper="0.0089" effort="5" velocity="0.05" />
+  </joint>
+  <joint name="manipulator_finger_joint2" type="prismatic">
+    <parent link="manipulator_gripper_shell" />
+    <child link="manipulator_finger2" />
+    <origin xyz="0 0 0.0543" rpy="0 0 0" />
+    <axis xyz="0 -1 0" />
+    <limit lower="0" upper="0.0089" effort="5" velocity="0.05" />
   </joint>
 </robot>

Commit message: 完善扫描场景导入与AI场景查询并同步车辆配置模型
补充扫描场景注册、删除与解码，增加只读场景查询及上下文缓存，完善全细节模型预览，并保存当前车辆导出配置和网格。相关回归测试112项通过，未纳入密钥、专利及软著材料。

File: ros2_ws/src/agribot_vehicle_description/generated/ackermann_current/urdf/ackermann_current.urdf.xacro (robot description, xacro)
@@ -28,5 +28,5 @@
   </link>
   <joint name="imu_mount_joint" type="fixed">
-    <origin xyz="0.142499953508 1.09291818262e-07 0.142997741699" rpy="0.000572424090933 -0.00913954898715 -2.61600916929e-06" />
+    <origin xyz="0.142499983311 5.68556153269e-08 0.142999649048" rpy="0.000572423974518 -0.00913954898715 -2.61600075646e-06" />
     <parent link="base_link" />
     <child link="imu_link" />
@@ -40,5 +40,5 @@
   </link>
   <joint name="lidar_mount_joint" type="fixed">
-    <origin xyz="0.479999929667 7.1564620896e-08 0.232997894287" rpy="-0.00764848804101 -0.00183566054329 7.01999897501e-06" />
+    <origin xyz="0.479999959469 3.54528566504e-08 0.232999801636" rpy="-0.00764848850667 -0.00183566124178 7.020000794e-06" />
     <parent link="base_link" />
     <child link="lidar_link" />
@@ -52,5 +52,5 @@
   </link>
   <joint name="right_camera_mount_joint" type="fixed">
-    <origin xyz="0.575500011444 9.52900123252e-08 0.153997421265" rpy="0 3.54046791884e-10 0" />
+    <origin xyz="0.575500011444 4.62625813213e-08 0.153999328613" rpy="0 0 0" />
     <parent link="base_link" />
     <child link="right_camera_link" />
@@ -58,5 +58,5 @@
   <link name="right_camera_optical_frame" />
   <joint name="right_camera_measurement_joint" type="fixed">
-    <origin xyz="8.74736727496e-09 9.52900123252e-08 -1.90754212781e-06" rpy="-1.57079637051 0 -1.57079637051" />
+    <origin xyz="2.5449002905e-09 4.62625813213e-08 0" rpy="-1.57079637051 0 -1.57079637051" />
     <parent link="right_camera_link" />
     <child link="right_camera_optical_frame" />
@@ -70,5 +70,5 @@
   </link>
   <joint name="rtk_master_mount_joint" type="fixed">
-    <origin xyz="0.142499923706 0.295258581638 0.784757614136" rpy="0 3.54046791884e-10 0" />
+    <origin xyz="0.142499953508 0.295258522034 0.784759521484" rpy="0 0 0" />
     <parent link="base_link" />
     <child link="rtk_link" />
@@ -77,5 +77,5 @@
   </link>
   <joint name="rtk_secondary_mount_joint" type="fixed">
-    <origin xyz="0.142499923706 -0.295258373022 0.784757614136" rpy="0 3.54046791884e-10 0" />
+    <origin xyz="0.142499953508 -0.295258462429 0.784759521484" rpy="0 0 0" />
     <parent link="base_link" />
     <child link="rtk_secondary_link" />
@@ -83,5 +83,5 @@
   <link name="front_left_steering_link" />
   <joint name="front_left_steering_joint" type="revolute">
-    <origin xyz="0.525849163532 0.294998288155 0.000398635689635" rpy="0 0 0" />
+    <origin xyz="0.52584695816 0.294999092817 0.00139999389648" rpy="0 0 0" />
     <parent link="base_link" />
     <child link="front_left_steering_link" />
@@ -110,5 +110,5 @@
   <link name="front_right_steering_link" />
   <joint name="front_right_steering_joint" type="revolute">
-    <origin xyz="0.527325689793 -0.294998109341 -0.000999450916424" rpy="0 0 0" />
+    <origin xyz="0.527324318886 -0.29499900341 0.00139999389648" rpy="0 0 0" />
     <parent link="base_link" />
     <child link="front_right_steering_link" />
@@ -149,5 +149,5 @@
   </link>
   <joint name="rear_left_wheel_joint" type="continuous">
-    <origin xyz="3.90425213936e-07 0.294999241829 0.000696182192769" rpy="0 0 0" />
+    <origin xyz="-3.08463832255e-08 0.294999986887 0" rpy="0 0 0" />
     <parent link="base_link" />
     <child link="rear_left_wheel_link" />
@@ -168,5 +168,5 @@
   </link>
   <joint name="rear_right_wheel_joint" type="continuous">
-    <origin xyz="-4.17683509113e-07 -0.294999063015 -0.00069999700645" rpy="0 0 0" />
+    <origin xyz="-2.36684734034e-08 -0.294999957085 -1.90734863281e-06" rpy="0 0 0" />
     <parent link="base_link" />
     <child link="rear_right_wheel_link" />
@@ -286,5 +286,5 @@
     <parent link="base_link" />
     <child link="manipulator_link_base" />
-    <origin xyz="0.2527782023 0.0006425103056 0.1394004822" rpy="0.002361407736 0.003225819673 6.398016922e-06" />
+    <origin xyz="0.2523272038 0.0009719826048 0.14021492" rpy="0 2.384185791e-07 1.131907794e-07" />
   </joint>
   <joint name="manipulator_joint1" type="revolute">
